File: MF68+10/MF68+10.kicad_pcb (KiCad board)
At the start: 2 copper layers, 370.5 x 94.4 mm, 171 parts, among them U1 Teensy_3.2, U2 AN32183A

Commit message: stitched ground planes
Parts:
- added REF**: GND Via, Cherry:GNDVia, F.Cu at (118.6, 64.8)
- added REF**: GND Via, Cherry:GNDVia, F.Cu at (74.9, 104.8)
- added REF**: GND Via, Cherry:GNDVia, F.Cu at (172.1, 85.7)
- added REF**: GND Via, Cherry:GNDVia, F.Cu at (191.1, 85.7)
- added REF**: GND Via, Cherry:GNDVia, F.Cu at (210.2, 85.7)
- added REF**: GND Via, Cherry:GNDVia, F.Cu at (229.2, 85.7)
- added REF**: GND Via, Cherry:GNDVia, F.Cu at (248.3, 85.1)
- added REF**: GND Via, Cherry:GNDVia, F.Cu at (267.3, 85.7)
- added REF**: GND Via, Cherry:GNDVia, F.Cu at (286.4, 85.7)
- added REF**: GND Via, Cherry:GNDVia, F.Cu at (148.6, 104.1)
- added REF**: GND Via, Cherry:GNDVia, F.Cu at (361.9, 28.6)
- added REF**: GND Via, Cherry:GNDVia, F.Cu at (157.7, 47.6)
- added REF**: GND Via, Cherry:GNDVia, F.Cu at (362.6, 47.6)
- added REF**: GND Via, Cherry:GNDVia, F.Cu at (358.8, 47.6)
- added REF**: GND Via, Cherry:GNDVia, F.Cu at (334.0, 47.6)
- added REF**: GND Via, Cherry:GNDVia, F.Cu at (309.9, 47.6)
- added REF**: GND Via, Cherry:GNDVia, F.Cu at (279.4, 28.6)
- added REF**: GND Via, Cherry:GNDVia, F.Cu at (260.4, 28.6)
- added REF**: GND Via, Cherry:GNDVia, F.Cu at (108.0, 28.6)
- added REF**: GND Via, Cherry:GNDVia, F.Cu at (127.0, 28.6)
- added REF**: GND Via, Cherry:GNDVia, F.Cu at (146.1, 28.6)
- added REF**: GND Via, Cherry:GNDVia, F.Cu at (165.7, 28.6)
- added REF**: GND Via, Cherry:GNDVia, F.Cu at (74.9, 77.2)
- added REF**: GND Via, Cherry:GNDVia, F.Cu at (184.8, 28.6)
- added REF**: GND Via, Cherry:GNDVia, F.Cu at (222.9, 28.6)
- added REF**: GND Via, Cherry:GNDVia, F.Cu at (203.8, 28.6)
- added REF**: GND Via, Cherry:GNDVia, F.Cu at (252.7, 47.6)
- added REF**: GND Via, Cherry:GNDVia, F.Cu at (271.8, 47.8)
- added REF**: GND Via, Cherry:GNDVia, F.Cu at (295.3, 66.7)
- added REF**: GND Via, Cherry:GNDVia, F.Cu at (276.9, 66.7)
- added REF**: GND Via, Cherry:GNDVia, F.Cu at (257.8, 66.7)
- added REF**: GND Via, Cherry:GNDVia, F.Cu at (238.8, 66.7)
- added REF**: GND Via, Cherry:GNDVia, F.Cu at (219.7, 66.7)
- added REF**: GND Via, Cherry:GNDVia, F.Cu at (128.0, 75.4)
- added REF**: GND Via, Cherry:GNDVia, F.Cu at (200.7, 66.7)
- added REF**: GND Via, Cherry:GNDVia, F.Cu at (181.6, 66.7)
- added REF**: GND Via, Cherry:GNDVia, F.Cu at (162.6, 66.7)
- added REF**: GND Via, Cherry:GNDVia, F.Cu at (139.1, 47.6)
- added REF**: GND Via, Cherry:GNDVia, F.Cu at (48.3, 66.7)
- added REF**: GND Via, Cherry:GNDVia, F.Cu at (48.3, 85.7)
- added REF**: GND Via, Cherry:GNDVia, F.Cu at (48.3, 104.8)
- added REF**: GND Via, Cherry:GNDVia, F.Cu at (121.9, 104.8)
- added REF**: GND Via, Cherry:GNDVia, F.Cu at (105.4, 66.0)
- added REF**: GND Via, Cherry:GNDVia, F.Cu at (143.5, 66.7)
- added REF**: GND Via, Cherry:GNDVia, F.Cu at (144.0, 75.2)
- added REF**: GND Via, Cherry:GNDVia, F.Cu at (153.0, 85.7)
- added REF**: GND Via, Cherry:GNDVia, F.Cu at (134.0, 85.7)
- added REF**: GND Via, Cherry:GNDVia, F.Cu at (114.9, 85.7)
- added REF**: GND Via, Cherry:GNDVia, F.Cu at (100.3, 47.6)
- added REF**: GND Via, Cherry:GNDVia, F.Cu at (76.8, 47.6)
- added REF**: GND Via, Cherry:GNDVia, F.Cu at (48.3, 47.6)
- added REF**: GND Via, Cherry:GNDVia, F.Cu at (220.6, 50.2)
- added REF**: GND Via, Cherry:GNDVia, F.Cu at (215.9, 47.5)
- added REF**: GND Via, Cherry:GNDVia, F.Cu at (334.1, 47.5)
- added REF**: GND Via, Cherry:GNDVia, F.Cu at (382.6, 47.5)
- added REF**: GND Via, Cherry:GNDVia, F.Cu at (159.5, 75.4)
- added REF**: GND Via, Cherry:GNDVia, F.Cu at (286.6, 107.2)
- added REF**: GND Via, Cherry:GNDVia, F.Cu at (241.1, 109.5)
- added REF**: GND Via, Cherry:GNDVia, F.Cu at (215.4, 106.8)
- added REF**: GND Via, Cherry:GNDVia, F.Cu at (188.0, 104.8)
- added REF**: GND Via, Cherry:GNDVia, F.Cu at (218.5, 96.5)
- added REF**: GND Via, Cherry:GNDVia, F.Cu at (226.0, 95.0)
- added REF**: GND Via, Cherry:GNDVia, F.Cu at (387.6, 84.5)
- added REF**: GND Via, Cherry:GNDVia, F.Cu at (397.6, 75.5)
- added REF**: GND Via, Cherry:GNDVia, F.Cu at (398.1, 93.0)
- added REF**: GND Via, Cherry:GNDVia, F.Cu at (397.6, 25.2)
- added REF**: GND Via, Cherry:GNDVia, F.Cu at (393.6, 85.7)
- added REF**: GND Via, Cherry:GNDVia, F.Cu at (372.4, 74.2)
- added REF**: GND Via, Cherry:GNDVia, F.Cu at (372.4, 63.0)
- added REF**: GND Via, Cherry:GNDVia, F.Cu at (372.4, 59.0)
- added REF**: GND Via, Cherry:GNDVia, F.Cu at (379.1, 74.2)
- added REF**: GND Via, Cherry:GNDVia, F.Cu at (380.9, 59.0)
- added REF**: GND Via, Cherry:GNDVia, F.Cu at (397.6, 59.0)
- added REF**: GND Via, Cherry:GNDVia, F.Cu at (266.8, 36.8)
- added REF**: GND Via, Cherry:GNDVia, F.Cu at (291.2, 36.8)
- added REF**: GND Via, Cherry:GNDVia, F.Cu at (351.0, 36.0)
- added REF**: GND Via, Cherry:GNDVia, F.Cu at (298.2, 28.8)
- added REF**: GND Via, Cherry:GNDVia, F.Cu at (74.9, 85.7)
- added REF**: GND Via, Cherry:GNDVia, F.Cu at (318.5, 28.8)
- added REF**: GND Via, Cherry:GNDVia, F.Cu at (238.0, 109.5)
- added REF**: GND Via, Cherry:GNDVia, F.Cu at (290.8, 47.8)
- added REF**: GND Via, Cherry:GNDVia, F.Cu at (303.0, 84.8)
- added REF**: GND Via, Cherry:GNDVia, F.Cu at (326.0, 89.2)
- added REF**: GND Via, Cherry:GNDVia, F.Cu at (292.0, 96.2)
- added REF**: GND Via, Cherry:GNDVia, F.Cu at (307.8, 109.5)
- added REF**: GND Via, Cherry:GNDVia, F.Cu at (336.0, 109.5)
- added REF**: GND Via, Cherry:GNDVia, F.Cu at (318.2, 76.8)
- added REF**: GND Via, Cherry:GNDVia, F.Cu at (74.9, 66.7)
- added REF**: GND Via, Cherry:GNDVia, F.Cu at (246.8, 97.2)
- added REF**: GND Via, Cherry:GNDVia, F.Cu at (252.2, 97.2)
- added REF**: GND Via, Cherry:GNDVia, F.Cu at (48.3, 28.6)
- added REF**: GND Via, Cherry:GNDVia, F.Cu at (73.7, 28.6)
- renumbered REF** to GND
Connections:
- GND pad 1: (no net) -> GND
- REF** pad 1: (no net) -> GND (x5)
Routing:
- net Z7: track 617.0 -> 564.7 mm
- net Z6: track 760.9 -> 778.2 mm, vias 2 -> 3
- net C1: track 517.4 -> 525.7 mm
- net Z4: track 705.7 -> 713.9 mm
- net GND: track 104.4 -> 111.6 mm, vias 5 -> 6
- net Z1: track 500.6 -> 507.2 mm
- net Z5: track 551.5 -> 545.4 mm
- net R3: track 361.3 -> 366.1 mm
- net C2: track 492.0 -> 496.5 mm
- net C8: track 379.0 -> 382.2 mm
- net R5: track 334.7 -> 337.9 mm
- net C3: track 497.0 -> 494.1 mm
- net Z9: track 545.3 -> 547.7 mm
- net Z10: track 149.5 -> 151.2 mm
- net Z2: track 664.8 -> 663.1 mm
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