File: 103key-project/103key.sch (KiCad schematic (older format))
At the start: 207 parts, among them U1 Teensy_3.2

Commit message: Changed key matrix to 10x11 to free up 3 teensy pins
Connections:
- net C1: now also SW_2_76.SW1, SW_5_60.SW1, SW_8_40.SW1, SW_Scroll_2.SW1, SW_X3Y3_20.SW1
- net C10: now also SW_Del_57.SW1, SW_Ins_37.SW1, SW_PgDn_58.SW1, SW_PgUp_38.SW1; no longer SW_B_84.SW1, SW_G_67.SW1, SW_T_48.SW1, SW_Win_99.SW1, SW_X11Y3_28.SW1
- net C2: now also SW_3_77.SW1, SW_6_61.SW1, SW_9_41.SW1, SW_Ctrl_94.SW1, SW_Enter_78.SW1, SW_Esc_4.SW1, SW_Pause_3.SW1, SW_X4Y3_21.SW1, SW_X4Y7_93.SW1, SW_X5Y3_22.SW1, SW_X5Y4_42.SW1; no longer SW_2_76.SW1, SW_5_60.SW1, SW_8_40.SW1, SW_Scroll_2.SW1, SW_X3Y3_20.SW1
- net C3: now also SW_A_63.SW1, SW_Caps_62.SW1, SW_F1_5.SW1, SW_F2_6.SW1, SW_Q_44.SW1, SW_Shift_79.SW1, SW_Tab_43.SW1, SW_Win_95.SW1, SW_X6Y3_23.SW1, SW_X7Y3_24.SW1, SW_Z_80.SW1; no longer SW_3_77.SW1, SW_6_61.SW1, SW_9_41.SW1, SW_Pause_3.SW1, SW_X4Y3_21.SW1, SW_X4Y7_93.SW1
- net C4: now also SW_Alt_96.SW1, SW_C_82.SW1, SW_D_65.SW1, SW_E_46.SW1, SW_F3_7.SW1, SW_F4_8.SW1, SW_S_64.SW1, SW_W_45.SW1, SW_X8Y3_25.SW1, SW_X9Y3_26.SW1, SW_X_81.SW1; no longer SW_Enter_78.SW1, SW_X5Y3_22.SW1, SW_X5Y4_42.SW1
- net C5: now also SW_B_84.SW1, SW_F5_9.SW1, SW_F6_10.SW1, SW_F_66.SW1, SW_G_67.SW1, SW_R_47.SW1, SW_T_48.SW1, SW_V_83.SW1, SW_X10Y3_27.SW1, SW_X10Y7_97.SW1, SW_X11Y3_28.SW1; no longer SW_Caps_62.SW1, SW_Ctrl_94.SW1, SW_Esc_4.SW1, SW_Shift_79.SW1, SW_Tab_43.SW1, SW_X6Y3_23.SW1
- net C6: now also SW_Alt_98.SW1, SW_F7_11.SW1, SW_F8_12.SW1, SW_H_68.SW1, SW_J_69.SW1, SW_M_86.SW1, SW_N_85.SW1, SW_U_50.SW1, SW_X12Y3_29.SW1, SW_X13Y3_30.SW1, SW_Y_49.SW1; no longer SW_A_63.SW1, SW_F1_5.SW1, SW_Q_44.SW1, SW_Win_95.SW1, SW_X7Y3_24.SW1, SW_Z_80.SW1
- net C7: now also SW_F10_14.SW1, SW_F9_13.SW1, SW_I_51.SW1, SW_K_70.SW1, SW_L_71.SW1, SW_O_52.SW1, SW_Win_99.SW1, SW_X14Y3_31.SW1, SW_X15Y3_32.SW1, SW_X15Y6_87.SW1, SW_X16Y6_88.SW1; no longer SW_Alt_96.SW1, SW_F2_6.SW1, SW_S_64.SW1, SW_W_45.SW1, SW_X8Y3_25.SW1, SW_X_81.SW1
- net C8: now also SW_F11_15.SW1, SW_F12_16.SW1, SW_Menu_100.SW1, SW_P_53.SW1, SW_Shift_90.SW1, SW_X16Y3_33.SW1, SW_X17Y3_34.SW1, SW_X17Y4_54.SW1, SW_X17Y5_72.SW1, SW_X17Y6_89.SW1, SW_X18Y5_73.SW1; no longer SW_C_82.SW1, SW_D_65.SW1, SW_E_46.SW1, SW_F3_7.SW1, SW_X10Y7_97.SW1, SW_X9Y3_26.SW1
- net C9: now also SW_Backspace_36.SW1, SW_End_18.SW1, SW_Enter_74.SW1, SW_Home_17.SW1, SW_X18Y3_35.SW1, SW_X18Y4_55.SW1, SW_X19Y4_56.SW1, SW_X20Y7_101.SW1, SW_X21Y6_91.SW1, SW_X21Y7_102.SW1, SW_X22Y7_103.SW1; no longer SW_Alt_98.SW1, SW_F4_8.SW1, SW_F_66.SW1, SW_R_47.SW1, SW_V_83.SW1, SW_X10Y3_27.SW1
- net R1: now also D17.1 (K); no longer D10.1 (K), D12.1 (K), D14.1 (K), D16.1 (K), D2.1 (K), D4.1 (K), D6.1 (K), D8.1 (K)
- net R2: now also D10.1 (K), D12.1 (K), D14.1 (K), D16.1 (K), D18.1 (K), D2.1 (K), D4.1 (K), D6.1 (K), D8.1 (K); no longer D19.1 (K), D20.1 (K), D21.1 (K), D22.1 (K), D23.1 (K), D24.1 (K), D25.1 (K), D26.1 (K), D27.1 (K), D28.1 (K), D29.1 (K), D30.1 (K), D31.1 (K), D32.1 (K), D33.1 (K), D34.1 (K), D35.1 (K), D36.1 (K)
- net R3: now also D19.1 (K), D21.1 (K), D23.1 (K), D25.1 (K), D27.1 (K), D29.1 (K), D31.1 (K), D33.1 (K), D35.1 (K), D37.1 (K); no longer D39.1 (K), D40.1 (K), D41.1 (K), D42.1 (K), D43.1 (K), D44.1 (K), D45.1 (K), D46.1 (K), D47.1 (K), D48.1 (K), D49.1 (K), D50.1 (K), D51.1 (K), D52.1 (K), D53.1 (K), D54.1 (K), D55.1 (K), D56.1 (K)
- net R4: now also D20.1 (K), D22.1 (K), D24.1 (K), D26.1 (K), D28.1 (K), D30.1 (K), D32.1 (K), D34.1 (K), D36.1 (K), D38.1 (K), U1.10 (10(CS)(TX2)); no longer D57.1 (K), D59.1 (K), D60.1 (K), D61.1 (K), D62.1 (K), D63.1 (K), D64.1 (K), D65.1 (K), D66.1 (K), D67.1 (K), D68.1 (K), D69.1 (K), D70.1 (K), D71.1 (K), D72.1 (K), D73.1 (K), D74.1 (K), D78.1 (K), U1.23 (23/A9)
- net R5: now also D39.1 (K), D41.1 (K), D43.1 (K), D45.1 (K), D47.1 (K), D49.1 (K), D51.1 (K), D53.1 (K), D55.1 (K), D57.1 (K), U1.9 (9(RX2)); no longer D58.1 (K), D75.1 (K), D76.1 (K), D77.1 (K), D79.1 (K), D80.1 (K), D81.1 (K), D82.1 (K), D83.1 (K), D84.1 (K), D85.1 (K), D86.1 (K), D87.1 (K), D88.1 (K), D89.1 (K), D90.1 (K), D91.1 (K), U1.22 (22/A8)
- net R6: now also D40.1 (K), D42.1 (K), D44.1 (K), D46.1 (K), D48.1 (K), D50.1 (K), D52.1 (K), D54.1 (K), D56.1 (K), D58.1 (K), U1.8 (8(TX3)); no longer D100.1 (K), D101.1 (K), D102.1 (K), D103.1 (K), D17.1 (K), D18.1 (K), D37.1 (K), D38.1 (K), D92.1 (K), D93.1 (K), D94.1 (K), D95.1 (K), D96.1 (K), D97.1 (K), D98.1 (K), D99.1 (K), U1.21 (21/A7)
- removed net C11: SW_F5_9.SW1, SW_H_68.SW1, SW_Menu_100.SW1, SW_N_85.SW1, SW_X12Y3_29.SW1, SW_Y_49.SW1, U1.5
- removed net C12: SW_F6_10.SW1, SW_J_69.SW1, SW_M_86.SW1, SW_U_50.SW1, SW_X13Y3_30.SW1, SW_X20Y7_101.SW1, U1.6
- removed net C13: SW_F7_11.SW1, SW_I_51.SW1, SW_K_70.SW1, SW_X14Y3_31.SW1, SW_X15Y6_87.SW1, SW_X21Y7_102.SW1, U1.7 (7(RX3))
- removed net C14: SW_F8_12.SW1, SW_L_71.SW1, SW_O_52.SW1, SW_X15Y3_32.SW1, SW_X16Y6_88.SW1, SW_X22Y7_103.SW1, U1.8 (8(TX3))
- removed net C15: SW_F9_13.SW1, SW_Ins_37.SW1, SW_P_53.SW1, SW_X16Y3_33.SW1, SW_X17Y5_72.SW1, SW_X17Y6_89.SW1, U1.9 (9(RX2))
- removed net C16: SW_F10_14.SW1, SW_PgUp_38.SW1, SW_Shift_90.SW1, SW_X17Y3_34.SW1, SW_X17Y4_54.SW1, SW_X18Y5_73.SW1, U1.10 (10(CS)(TX2))
- removed net C17: SW_Enter_74.SW1, SW_F11_15.SW1, SW_Home_17.SW1, SW_X18Y3_35.SW1, SW_X18Y4_55.SW1, SW_X21Y6_91.SW1, U1.11 (11(DOUT))
- removed net C18: SW_Backspace_36.SW1, SW_Del_57.SW1, SW_End_18.SW1, SW_F12_16.SW1, SW_PgDn_58.SW1, SW_X19Y4_56.SW1, U1.12 (12(DIN))
- new net R10: D102.1 (K), D76.1 (K), D80.1 (K), D82.1 (K), D84.1 (K), D86.1 (K), D88.1 (K), D90.1 (K), D94.1 (K), U1.11 (11(DOUT))
- new net R11: D100.1 (K), D103.1 (K), D92.1 (K), D93.1 (K), D95.1 (K), D96.1 (K), D97.1 (K), D98.1 (K), D99.1 (K), U1.12 (12(DIN))
- new net R7: D59.1 (K), D61.1 (K), D62.1 (K), D64.1 (K), D66.1 (K), D68.1 (K), D70.1 (K), D72.1 (K), D74.1 (K), U1.7 (7(RX3))
- new net R8: D60.1 (K), D63.1 (K), D65.1 (K), D67.1 (K), D69.1 (K), D71.1 (K), D73.1 (K), D78.1 (K), D91.1 (K), U1.6
- new net R9: D101.1 (K), D75.1 (K), D77.1 (K), D79.1 (K), D81.1 (K), D83.1 (K), D85.1 (K), D87.1 (K), D89.1 (K), U1.5
- new net RBG_1: U1.23 (23/A9)
- new net RGB_2: U1.22 (22/A8)
- new net RGB_3: U1.21 (21/A7)
