File: LFK78/LFK78.kicad_pcb (KiCad board)
At the start: 2 copper layers, 367.8 x 92.5 mm, 517 parts, among them J1 USB_OTG, SW1 SW_RST, U1 ATMEGA32U4RC-A, U2 IS31FL3731, U3 IS31FL3731, X1 16Mhz, X2 PiezoelectricCrystal-TwoElect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

Commit message: LFK78 RevC addedd
Parts:
- removed the REF** at (191.0, 96.2)
- removed the REF** at (128.4, 84.5)
- removed the REF** at (304.7, 22.4)
- removed the REF** at (277.7, 22.6)
- removed the REF** at (286.2, 22.1)
- removed the REF** at (259.6, 22.6)
- removed the REF** at (240.6, 22.8)
- removed the REF** at (221.1, 22.6)
- removed the REF** at (182.2, 22.3)
- removed the REF** at (159.8, 21.5)
- removed the REF** at (143.0, 21.9)
- removed the REF** at (381.5, 105.3)
- removed the REF** at (377.7, 105.3)
- removed the REF** at (366.7, 108.1)
- removed the REF** at (382.9, 85.1)
- removed the REF** at (386.7, 90.8)
- removed the REF** at (367.3, 72.7)
- removed the REF** at (373.4, 68.9)
- removed the REF** at (367.0, 68.9)
- removed the REF** at (340.3, 72.3)
- removed the REF** at (343.9, 71.0)
- removed the REF** at (343.9, 67.8)
- removed the REF** at (346.2, 62.5)
- removed the REF** at (343.5, 62.5)
- removed the REF** at (343.5, 57.1)
- removed the REF** at (346.1, 57.1)
- removed the REF** at (373.3, 72.5)
- removed the REF** at (373.6, 60.1)
- removed the REF** at (244.5, 105.5)
- removed the REF** at (384.3, 31.3)
- removed the REF** at (376.8, 21.6)
- removed the REF** at (360.2, 31.9)
- removed the REF** at (338.4, 48.2)
- removed the REF** at (345.2, 40.8)
- removed the REF** at (295.7, 34.5)
- removed the REF** at (303.7, 47.7)
- removed the REF** at (232.0, 105.5)
- removed the REF** at (319.3, 53.5)
- removed the REF** at (329.0, 52.9)
- removed the REF** at (328.9, 46.7)
- removed the REF** at (323.9, 46.7)
- removed the REF** at (33.5, 83.0)
- removed the REF** at (254.0, 109.5)
- removed the REF** at (322.0, 74.9)
- removed the REF** at (321.9, 68.8)
- removed the REF** at (318.5, 74.9)
- removed the REF** at (316.7, 79.5)
- removed the REF** at (301.0, 66.0)
- removed the REF** at (285.9, 75.2)
- removed the REF** at (304.5, 71.1)
- removed the REF** at (304.3, 79.2)
- removed the REF** at (301.8, 90.7)
- removed the REF** at (304.5, 90.7)
- removed the REF** at (315.0, 85.3)
- removed the REF** at (321.6, 90.4)
- removed the REF** at (321.7, 82.5)
- removed the REF** at (314.9, 90.7)
- removed the REF** at (308.1, 90.7)
- removed the REF** at (328.9, 110.5)
- removed the REF** at (316.2, 104.4)
- removed the REF** at (347.1, 67.4)
- removed the REF** at (354.8, 67.8)
- removed the REF** at (350.6, 67.5)
- removed the REF** at (204.1, 62.3)
- removed the REF** at (202.5, 23.3)
- removed the REF** at (190.2, 22.7)
- removed the REF** at (190.3, 30.0)
- removed the REF** at (115.3, 27.5)
- removed the REF** at (133.7, 27.8)
- removed the REF** at (171.3, 110.8)
- removed the REF** at (151.7, 110.9)
- removed the REF** at (140.9, 105.2)
- removed the REF** at (171.3, 99.7)
- removed the REF** at (151.7, 100.0)
- removed the REF** at (136.8, 99.7)
- removed the REF** at (119.1, 110.1)
- removed the REF** at (80.2, 90.6)
- removed the REF** at (85.6, 85.6)
- removed the REF** at (171.3, 96.2)
- removed the REF** at (101.5, 57.3)
- removed the REF** at (94.3, 57.3)
- removed the REF** at (114.7, 72.3)
- removed the REF** at (116.6, 85.7)
- removed the REF** at (113.1, 80.4)
- removed the REF** at (105.4, 73.0)
- removed the REF** at (105.7, 79.9)
- removed the REF** at (108.1, 80.1)
- removed the REF** at (108.5, 83.4)
- removed the REF** at (100.5, 83.0)
- removed the REF** at (97.3, 83.6)
- removed the REF** at (102.0, 91.1)
- removed the REF** at (107.6, 92.2)
- removed the REF** at (140.7, 96.3)
- removed the REF** at (110.2, 103.1)
- removed the REF** at (99.1, 71.1)
- removed the REF** at (193.9, 56.9)
- removed the REF** at (80.3, 57.4)
- removed the REF** at (34.0, 25.5)
- removed the REF** at (80.3, 47.8)
- removed the REF** at (122.0, 21.5)
- removed the REF** at (97.7, 103.9)
- removed the REF** at (97.8, 110.0)
- removed the REF** at (349.9, 42.0)
- removed the REF** at (361.7, 41.9)
- removed the REF** at (355.1, 47.2)
- removed the REF** at (350.5, 47.2)
- removed the REF** at (361.7, 47.2)
- removed the REF** at (345.9, 33.5)
- removed the REF** at (365.3, 23.4)
- removed the REF** at (348.0, 71.9)
- removed the REF** at (359.7, 75.2)
- removed the REF** at (348.0, 75.6)
- removed the REF** at (359.6, 68.0)
- removed the REF** at (358.0, 63.7)
- removed the REF** at (286.0, 27.7)
- removed the REF** at (206.2, 111.0)
- removed the REF** at (217.5, 110.0)
- removed the REF** at (363.2, 71.9)
- removed the REF** at (339.5, 90.1)
- removed the REF** at (359.7, 90.2)
- removed the REF** at (360.4, 85.3)
- removed the REF** at (339.2, 85.1)
- removed the REF** at (394.3, 97.0)
- removed the REF** at (172.1, 85.7)
- removed the REF** at (229.2, 85.7)
- removed the REF** at (248.3, 85.1)
- removed the REF** at (334.0, 47.6)
- removed the REF** at (314.9, 82.4)
- removed the REF** at (295.2, 66.0)
- removed the REF** at (48.5, 85.7)
- removed the REF** at (48.3, 104.8)
- removed the REF** at (335.2, 76.2)
- removed the REF** at (124.8, 103.9)
- removed the REF** at (105.4, 66.0)
- removed the REF** at (153.0, 85.7)
- removed the REF** at (288.9, 105.9)
- removed the REF** at (217.9, 98.3)
- removed the REF** at (228.0, 110.0)
- removed the REF** at (337.9, 76.2)
- removed the REF** at (48.3, 28.6)
- removed the REF** at (228.0, 99.5)
- removed the REF** at (76.9, 27.9)
- removed the REF** at (354.4, 27.4)
- removed the REF** at (65.5, 22.0)
- removed the REF** at (254.0, 100.5)
- removed the REF** at (77.5, 106.0)
- removed the REF** at (76.8, 97.8)
- removed the REF** at (75.6, 22.9)
- removed the REF** at (186.9, 66.7)
- removed the REF** at (102.5, 21.5)
- removed the REF** at (109.0, 96.3)
- removed the REF** at (118.9, 96.3)
- removed the REF** at (106.9, 57.1)
- removed the REF** at (108.5, 66.0)
- removed the REF** at (197.0, 67.3)
- removed the REF** at (391.4, 73.2)
- removed the REF** at (363.3, 51.8)
- removed the REF** at (354.6, 51.7)
- removed the REF** at (350.6, 51.7)
- removed the REF** at (350.0, 57.3)
- removed the REF** at (351.9, 60.1)
- removed the REF** at (354.3, 90.2)
- removed the REF** at (349.2, 90.2)
- removed the REF** at (349.2, 85.7)
- removed the REF** at (335.3, 85.1)
- removed the REF** at (329.6, 69.2)
- removed the REF** at (329.6, 74.9)
- removed the REF** at (328.5, 84.6)
- removed the REF** at (117.5, 89.3)
- removed the REF** at (304.5, 85.1)
- removed the REF** at (273.1, 85.7)
- removed the REF** at (290.2, 85.7)
- removed the REF** at (282.6, 66.0)
- removed the REF** at (229.2, 52.7)
- removed the REF** at (239.4, 28.6)
- removed the REF** at (99.3, 80.6)
- removed the REF** at (234.3, 31.8)
- removed the REF** at (245.2, 45.7)
- removed the REF** at (285.6, 71.3)
- removed the REF** at (43.3, 38.3)
- removed the REF** at (132.4, 78.7)
- removed the REF** at (43.5, 25.5)
- removed the REF** at (85.3, 23.7)
- removed the REF** at (106.0, 47.9)
- removed the REF** at (390.1, 94.3)
- removed the REF** at (393.6, 86.6)
- removed the REF** at (392.1, 77.3)
- removed U1: ATMEGA32U4RC-A, Housings_QFP:TQFP-44_10x10mm_Pitch0.8mm
- removed the X2 at (238.4, 105.5)
- added ?: ALPS, Keyboard:ALPS, F.Cu at (57.1, 28.6)
- added ?: ALPS, Keyboard:ALPS, F.Cu at (57.1, 104.8)
- added ?: ALPS, Keyboard:ALPS, F.Cu at (38.1, 28.6)
- added ?: ALPS, Keyboard:ALPS, F.Cu at (57.1, 47.6)
- added ?: ALPS, Keyboard:ALPS, F.Cu at (38.1, 47.6)
- added ?: ALPS, Keyboard:ALPS, F.Cu at (38.0, 66.7)
- added ?: ALPS, Keyboard:ALPS, F.Cu at (57.1, 66.7)
- added ?: ALPS, Keyboard:ALPS, F.Cu at (57.1, 85.7)
- added ?: ALPS, Keyboard:ALPS, F.Cu at (38.1, 85.7)
- added ?: ALPS, Keyboard:ALPS, F.Cu at (38.1, 104.8)
- added C13: 1µF, Capacitors_SMD:C_0805, F.Cu at (214.4, 122.6)
- added D79: D, Diodes_SMD:SOD-123, B.Cu at (99.9, 81.0)
- added R12: 10KΩ, Resistors_SMD:R_0805, F.Cu at (214.4, 122.6)
- added REF**: MountingHole_6mm, Mounting_Holes:MountingHole_6mm, F.Cu at (100.0, 67.0)
- added REF**: MountingHole_6mm, Mounting_Holes:MountingHole_6mm, F.Cu at (90.4, 31.0)
- added REF**: MountingHole_6mm, Mounting_Holes:MountingHole_6mm, F.Cu at (95.2, 102.1)
- added REF**: MountingHole_6mm, Mounting_Holes:MountingHole_6mm, F.Cu at (238.1, 97.8)
- added REF**: MountingHole_6mm, Mounting_Holes:MountingHole_6mm, F.Cu at (381.0, 102.1)
- added REF**: MountingHole_6mm, Mounting_Holes:MountingHole_6mm, F.Cu at (381.0, 31.0)
- added REF**: MountingHole_6mm, Mounting_Holes:MountingHole_6mm, F.Cu at (242.8, 31.0)
- added REF**: GND Via, Keyboard:GNDVia-wRing, F.Cu at (62.0, 77.0)
- added REF**: GND Via, Keyboard:GNDVia-wRing, F.Cu at (80.5, 64.0)
- added STA: Stabilizer, Keyboard:CHERRY_PCB_200_STABILIZER_OUTLINE, F.Cu at (335.8, 66.7)
- added STA: Stabilizer, Keyboard:CHERRY_PCB_200_STABILIZER_OUTLINE, F.Cu at (331.0, 85.7)
- added STA: Stabilizer, Keyboard:CHERRY_PCB_200_STABILIZER_OUTLINE, F.Cu at (338.1, 28.6)
- added STA: Stabilizer, Keyboard:CHERRY_PCB_200_STABILIZER_OUTLINE, F.Cu at (92.9, 85.7)
- added SW_28: SW_28, Keyboard:MXALPS, F.Cu at (345.3, 57.1)
- added SW_41: SW_41, Keyboard:MXALPS, F.Cu at (323.9, 66.7)
- added SW_42: SW_42, Keyboard:MXALPS, F.Cu at (83.3, 85.7)
- added SW_55: SW_55, Keyboard:MXALPS_REVERSE_LED, F.Cu at (85.7, 104.8)
- added SW_56: SW_56, Keyboard:MXALPS, F.Cu at (111.9, 104.8)
- added SW_57: SW_57, Keyboard:MXALPS, F.Cu at (138.1, 104.8)
- added SW_58: SW_58, Keyboard:MXALPS, F.Cu at (214.3, 104.8)
- added SW_59: SW_59, Keyboard:MXALPS_REVERSE_LED, F.Cu at (290.5, 104.8)
- added SW_60: SW_60, Keyboard:MXALPS, F.Cu at (316.7, 104.8)
- added SW_AEK_1: SW_60, Keyboard:MXALPS, F.Cu at (288.1, 104.8)
- added SW_AEK_1: SW_60, Keyboard:MXALPS_REVERSE_LED, F.Cu at (314.3, 104.8)
- added SW_AEK_1: SW_60, Keyboard:MXALPS_REVERSE_LED, F.Cu at (319.1, 104.8)
- added SW_ISO_SLASH_79: MX_LED, Keyboard:MXALPS, F.Cu at (104.8, 85.7)
- added U4: IS31FL3731, Housings_SSOP:SSOP-28_5.3x10.2mm_Pitch0.65mm, F.Cu at (214.4, 122.6)
- C14: value 1µF -> 0.1µF
- D1, D10, D11, D12, D13, D14, D15, D16, D17, D18, D19, D2, D20, D21, D22, D23, D24, D25, D26, D27, D28, D29, D3, D30, D31, D32, D33, D34, D35, D36, D37, D38, D39, D4, D40, D41, D42, D43, D44, D45, D46, D47, D48, D49, D5, D50, D51, D52, D53, D54, D55, D56, D57, D58, D59, D6, D60, D61, D62, D63, D64, D65, D66, D67, D68, D69, D7, D70, D71, D72, D73, D74, D75, D76, D77, D78, D8, D9: footprint Diodes_ThroughHole:Diode_DO-35_SOD27_Horizontal_RM10 -> Diodes_SMD:SOD-123; moved to B.Cu
- R1: value 10KΩ -> 4.7KΩ
- R10: value 4.7KΩ -> 20KΩ; footprint Resistors_SMD:R_0805_HandSoldering -> Resistors_SMD:R_0805; moved to F.Cu
- R11: value 10KΩ -> 20KΩ
- R2: value 20KΩ -> 4.7KΩ
- R9: value 4.7KΩ -> 10KΩ; footprint Resistors_SMD:R_0805_HandSoldering -> Resistors_SMD:R_0805; moved to F.Cu
- SW_A_40, SW_Alt_71, SW_Alt_73, SW_B_59, SW_Backspace_16, SW_C_57, SW_CapStep_39, SW_Caps_39, SW_Ctrl_69, SW_D_42, SW_Del_35, SW_E_24, SW_Enter_51, SW_F10_68, SW_F1_1, SW_F2_2, SW_F3_19, SW_F4_20, SW_F5_37, SW_F6_38, SW_F7_52, SW_F8_53, SW_F9_67, SW_F_43, SW_G_44, SW_H_45, SW_I_29, SW_Ins_17, SW_J_46, SW_K_47, SW_L_48, SW_M_61, SW_Menu_75, SW_N_60, SW_O_30, SW_P_31, SW_PgDn_36, SW_PgUp_18, SW_Q_22, SW_R_25, SW_S_41, SW_Shift_54, SW_Shift_65, SW_T_26, SW_Tab_21, SW_U_28, SW_V_58, SW_W_23, SW_Win_70, SW_Win_74, SW_X10Y1_9, SW_X11Y1_10, SW_X12Y1_11, SW_X13Y1_12, SW_X13Y4_62, SW_X14Y1_13, SW_X14Y4_63, SW_X15Y1_14, SW_X15Y2_32, SW_X15Y3_49, SW_X15Y4_64, SW_X16Y1_15, SW_X16Y2_33, SW_X16Y3_50, SW_X17Y2_34, SW_X18Y5_76, SW_X19Y4_66, SW_X19Y5_77, SW_X20Y5_78, SW_X4Y1_3, SW_X5Y1_4, SW_X6Y1_5, SW_X7Y1_6, SW_X8Y1_7, SW_X8Y5_72, SW_X9Y1_8, SW_X_56, SW_Y_27, SW_Z_55: footprint Cherry:MXALPS_LED_PANEL -> Keyboard:MXALPS
- U2: value IS31FL3731 -> AT90USB1286; footprint Housings_SSOP:SSOP-28_5.3x10.2mm_Pitch0.65mm -> Housings_QFP:TQFP-64_14x14mm_Pitch0.8mm
- U3: moved to F.Cu
- moved U2 256.5 mm to (362.8, 66.5), turned to 270 degrees
- moved U3 120.5 mm to (214.4, 122.6), turned to 0 degrees
- moved R9 110.5 mm to (214.4, 122.6)
- moved R10 109.6 mm to (214.4, 122.6)
- moved D51 27.3 mm to (319.0, 61.8), turned to 270 degrees
- moved D39 25.8 mm to (78.0, 61.8), turned to 270 degrees
- moved C5 24.6 mm to (371.0, 56.7), turned to 180 degrees
- moved C1 23.4 mm to (98.0, 56.5)
- moved C2 23.4 mm to (98.0, 54.4)
- moved D65 23.2 mm to (325.8, 81.0)
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Connections:
- C15 pad 1: +5V -> Net-(C15-Pad1)
- D10 pad 1: R6 -> R1
- D11 pad 1: R6 -> R1
- D12 pad 1: R6 -> R1
- D13 pad 1: R6 -> R1
- D14 pad 1: R6 -> R1
- D15 pad 1: R6 -> R1
- D16 pad 1: R6 -> R1
- D17 pad 1: R10 -> R1
- D18 pad 1: R10 -> R1
- D19 pad 1: R2/SCK -> R2
- D20 pad 1: R2/SCK -> R2
- D21 pad 1: R2/SCK -> R2
- D22 pad 1: R2/SCK -> R2
- D23 pad 1: R2/SCK -> R2
- D24 pad 1: R2/SCK -> R2
- D25 pad 1: R2/SCK -> R2
- D26 pad 1: R2/SCK -> R2
- D27 pad 1: R7 -> R2
- D28 pad 1: R7 -> R2
- D29 pad 1: R7 -> R2
- D30 pad 1: R7 -> R2
- D31 pad 1: R7 -> R2
- D32 pad 1: R7 -> R2
- D33 pad 1: R7 -> R2
- D34 pad 1: R7 -> R2
- D35 pad 1: R10 -> R2
- D36 pad 1: R10 -> R2
- D37 pad 1: R3/MOSI -> R3
- D38 pad 1: R3/MOSI -> R3
- D39 pad 1: R3/MOSI -> R3
- D40 pad 1: R3/MOSI -> R3
- D41 pad 1: R3/MOSI -> R3
- D42 pad 1: R3/MOSI -> R3
- D43 pad 1: R3/MOSI -> R3
- D44 pad 1: R3/MOSI -> R3
- D45 pad 1: R8 -> R3
- D46 pad 1: R8 -> R3
- D47 pad 1: R8 -> R3
- D48 pad 1: R8 -> R3
- D49 pad 1: R8 -> R3
- D50 pad 1: R8 -> R3
- D51 pad 1: R8 -> R3
- D52 pad 1: R4/MISO -> R4
- D53 pad 1: R4/MISO -> R4
- D54 pad 1: R4/MISO -> R4
- D55 pad 1: R4/MISO -> R4
- D56 pad 1: R4/MISO -> R4
- D57 pad 1: R4/MISO -> R4
- D58 pad 1: R4/MISO -> R4
- D59 pad 1: R4/MISO -> R4
- D60 pad 1: R9 -> R4
- D61 pad 1: R9 -> R4
- D62 pad 1: R9 -> R4
- D63 pad 1: R9 -> R4
- D64 pad 1: R9 -> R4
- D65 pad 1: R9 -> R4
- D66 pad 1: R9 -> R4
- D75 pad 1: R10 -> R5
- D76 pad 1: R10 -> Net-(D76-Pad1)
- D77 pad 1: R10 -> R5
- D78 pad 1: R10 -> R5
- D9 pad 1: R6 -> R1
- R1 pad 1: Net-(R1-Pad1) -> +5V
- R1 pad 2: +5V -> LED_SDA
- R10 pad 1: +5V -> Net-(R10-Pad1)
- R10 pad 2: LED_SCL -> GND
- R11 pad 2: +5V -> GND
- R2 pad 1: Net-(R2-Pad1) -> +5V
- R2 pad 2: GND -> LED_SCL
- R9 pad 1: +5V -> Net-(R9-Pad1)
- R9 pad 2: LED_SDA -> +5V
- SW_Alt_73 pad SW1: C7 -> C13
- SW_B_59 pad SW1: C8 -> C9
- SW_Backspace_16 pad SW1: C8 -> C16
- SW_C_57 pad SW1: C6 -> C7
- SW_Del_35 pad SW1: C7 -> C17
- SW_Enter_51 pad SW1: C7 -> C15
- SW_H_45 pad SW1: C1 -> C9
- SW_I_29 pad SW1: C3 -> C11
- SW_Ins_17 pad SW1: C5 -> C17
- SW_J_46 pad SW1: C2 -> C10
- SW_K_47 pad SW1: C3 -> C11
- SW_L_48 pad SW1: C4 -> C12
- SW_M_61 pad SW1: C2 -> C11
- SW_Menu_75 pad SW1: C1 -> C15
- SW_N_60 pad SW1: C1 -> C10
- SW_O_30 pad SW1: C4 -> C12
- SW_P_31 pad SW1: C5 -> C13
- SW_PgDn_36 pad SW1: C8 -> C18
- SW_PgUp_18 pad SW1: C6 -> C18
- SW_Shift_65 pad SW1: C6 -> C15
- SW_U_28 pad SW1: C2 -> C10
- SW_V_58 pad SW1: C7 -> C8
- SW_Win_74 pad SW1: C8 -> C14
- SW_X10Y1_9 pad SW1: C1 -> C9
- SW_X11Y1_10 pad SW1: C2 -> C10
- SW_X12Y1_11 pad SW1: C3 -> C11
- SW_X13Y1_12 pad SW1: C4 -> C12
- SW_X13Y4_62 pad SW1: C3 -> C12
- SW_X14Y1_13 pad SW1: C5 -> C13
- SW_X14Y4_63 pad SW1: C4 -> C13
- SW_X15Y1_14 pad SW1: C6 -> C14
- SW_X15Y2_32 pad SW1: C6 -> C14
- SW_X15Y3_49 pad SW1: C5 -> C13
- SW_X15Y4_64 pad SW1: C5 -> C14
- SW_X16Y1_15 pad SW1: C7 -> C15
- SW_X16Y2_33 pad SW1: C7 -> C15
- SW_X16Y3_50 pad SW1: C6 -> C14
- SW_X17Y2_34 pad SW1: C8 -> C16
- SW_X18Y5_76 pad SW1: C2 -> C17
- SW_X19Y4_66 pad SW1: C7 -> C18
- SW_X19Y5_77 pad SW1: C3 -> C17
- SW_X20Y5_78 pad SW1: C4 -> C18
- SW_X8Y5_72 pad SW1: C6 -> C9
- SW_X_56 pad SW1: C5 -> C6
- SW_Y_27 pad SW1: C1 -> C9
- SW_Z_55 pad SW1: C4 -> C5
- U2 pad 1: L_CA9 -> C17
- U2 pad 10: L_CB4 -> Net-(U2-Pad10)
- U2 pad 11: L_CB5 -> SCK
- U2 pad 12: L_CB6 -> MOSI
- U2 pad 13: L_CB7 -> MISO
- U2 pad 14: L_CB8 -> Net-(U2-Pad14)
- U2 pad 15: L_CB9 -> PWM_RED
- U2 pad 16: Net-(C3-Pad1) -> PWM_GREEN
- U2 pad 17: Net-(U2-Pad17) -> PWM_BLUE
- U2 pad 18: GND -> Net-(U2-Pad18)
- U2 pad 19: LED_SDA -> Net-(U2-Pad19)
- U2 pad 2: +5V -> C18
- U2 pad 20: LED_SCL -> RST
- U2 pad 21: L_CA1 -> +5V
- U2 pad 22: L_CA2 -> GND
- U2 pad 23: L_CA3 -> Net-(C10-Pad1)
- U2 pad 24: L_CA4 -> Net-(C9-Pad1)
- U2 pad 25: L_CA5 -> LED_SCL
- U2 pad 26: L_CA6 -> LED_SDA
- U2 pad 27: L_CA7 -> Net-(U2-Pad27)
- U2 pad 28: L_CA8 -> Net-(U2-Pad28)
- U2 pad 3: Net-(R1-Pad1) -> +5V
- U2 pad 4: Net-(U2-Pad4) -> D-
- U2 pad 5: GND -> D+
- U2 pad 6: Net-(R2-Pad1) -> GND
- U2 pad 7: L_CB1 -> Net-(C11-Pad1)
- U2 pad 8: L_CB2 -> +5V
- U2 pad 9: L_CB3 -> Net-(U2-Pad9)
- U3 pad 1: R_CA9 -> L_CA9
- U3 pad 10: R_CB4 -> L_CB4
- U3 pad 11: R_CB5 -> L_CB5
- U3 pad 12: R_CB6 -> L_CB6
- U3 pad 13: R_CB7 -> L_CB7
- U3 pad 14: R_CB8 -> L_CB8
- U3 pad 15: R_CB9 -> L_CB9
- U3 pad 16: Net-(C16-Pad1) -> Net-(C3-Pad1)
- U3 pad 18: +5V -> GND
- U3 pad 21: R_CA1 -> L_CA1
- U3 pad 22: R_CA2 -> L_CA2
- U3 pad 23: R_CA3 -> L_CA3
- U3 pad 24: R_CA4 -> L_CA4
- U3 pad 25: R_CA5 -> L_CA5
- U3 pad 26: R_CA6 -> L_CA6
- U3 pad 27: R_CA7 -> L_CA7
- U3 pad 28: R_CA8 -> L_CA8
- U3 pad 3: Net-(R11-Pad1) -> Net-(R9-Pad1)
- U3 pad 6: Net-(R13-Pad1) -> Net-(R10-Pad1)
- U3 pad 7: R_CB1 -> L_CB1
- U3 pad 8: R_CB2 -> L_CB2
- U3 pad 9: R_CB3 -> L_CB3
Routing:
- net C5: track 663.5 -> 0.00 mm, vias 7 -> 0
- net C3: track 549.5 -> 0.00 mm, vias 11 -> 0
- net C1: track 521.1 -> 0.00 mm, vias 7 -> 0
- net C7: track 508.0 -> 0.00 mm, vias 8 -> 0
- net C6: track 500.7 -> 0.00 mm, vias 7 -> 0
- net C4: track 495.3 -> 0.00 mm, vias 6 -> 0
- net C2: track 471.0 -> 0.00 mm, vias 2 -> 0
- net C8: track 440.3 -> 0.03 mm, vias 7 -> 0
- net L_CB3: track 423.3 -> 0.00 mm, vias 7 -> 0
- net R3/MOSI: track 408.4 -> 0.00 mm, vias 3 -> 0
- net R_CB3: track 402.5 -> 0.00 mm, vias 9 -> 0
- net R_CA1: track 395.2 -> 0.00 mm, vias 3 -> 0
- net L_CB2: track 377.6 -> 0.00 mm, vias 9 -> 0
- net R4/MISO: track 369.6 -> 0.00 mm, vias 2 -> 0
- net R_CA4: track 367.3 -> 0.00 mm, vias 7 -> 0
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Other:
- net class Default: trace_width 0.381 -> 0.3048; via_dia 0.6096 -> 0.6858; via_drill 0.3048 -> 0.3302
- net class USB added: clearance 0.1524, trace_width 0.1524, via_dia 0.6858, via_drill 0.3302
- net class backlight added: clearance 0.1905, trace_width 0.254, via_dia 0.6858, via_drill 0.3302
- net class matrix added: clearance 0.1778, trace_width 0.2032, via_dia 0.6858, via_drill 0.3302
- net class power added: clearance 0.1905, trace_width 0.381, via_dia 0.6858, via_drill 0.3302
- net class underglow added: clearance 0.1905, trace_width 0.254, via_dia 0.6858, via_drill 0.3302
- rule trace_min: 0.254 -> 0.1524
- rule via_min_drill: 0.3048 -> 0.3302
- rule via_min_size: 0.6096 -> 0.6858
- board text added: "LFK78 RevC"
- board text added: "LFK78 RevC - ISO/ANSI"
- board text removed: "CENTER"
- board text removed: "LFK78 RevA"

Commit message: revC board completed with USB and mounting holes verified for VA68M case.
Parts:
- removed ? (x10): ALPS, Keyboard:ALPS
- removed C13: 1µF, Capacitors_SMD:C_0805
- removed D79: D, Diodes_SMD:SOD-123
- removed R12: 10KΩ, Resistors_SMD:R_0805
- removed the REF** at (100.0, 67.0)
- removed the REF** at (90.4, 31.0)
- removed the REF** at (95.2, 102.1)
- removed the REF** at (238.1, 97.8)
- removed the REF** at (381.0, 102.1)
- removed the REF** at (381.0, 31.0)
- removed the REF** at (242.8, 31.0)
- removed the REF** at (62.0, 77.0)
- removed the REF** at (80.5, 64.0)
- removed the REF** at (396.0, 34.0)
- removed STA (x4): Stabilizer, Keyboard:CHERRY_PCB_200_STABILIZER_OUTLINE
- removed SW_28: SW_28, Keyboard:MXALPS
- removed SW_41: SW_41, Keyboard:MXALPS
- removed SW_42: SW_42, Keyboard:MXALPS
- removed SW_55: SW_55, Keyboard:MXALPS_REVERSE_LED
- removed SW_56: SW_56, Keyboard:MXALPS
- removed SW_57: SW_57, Keyboard:MXALPS
- removed SW_58: SW_58, Keyboard:MXALPS
- removed SW_59: SW_59, Keyboard:MXALPS_REVERSE_LED
- removed SW_60, SW_AEK_1: SW_60, Keyboard:MXALPS
- removed SW_AEK_1 (x2): SW_60, Keyboard:MXALPS_REVERSE_LED
- removed SW_ISO_SLASH_79: MX_LED, Keyboard:MXALPS
- removed U4: IS31FL3731, Housings_SSOP:SSOP-28_5.3x10.2mm_Pitch0.65mm
- added CHERRY: MX, Cherry:CHERRY_PCB_200H_STABILIZER, F.Cu at (338.1, 28.6)
- added REF**: GND Via, Keyboard:GNDVia-wRing, F.Cu at (132.4, 78.7)
- added REF**: GND Via, Keyboard:GNDVia-wRing, F.Cu at (354.3, 90.2)
- added REF**: GND Via, Keyboard:GNDVia-wRing, F.Cu at (349.2, 90.2)
- added REF**: GND Via, Keyboard:GNDVia-wRing, F.Cu at (349.2, 85.7)
- added REF**: GND Via, Keyboard:GNDVia-wRing, F.Cu at (335.3, 85.1)
- added REF**: GND Via, Keyboard:GNDVia-wRing, F.Cu at (329.6, 69.2)
- added REF**: GND Via, Keyboard:GNDVia-wRing, F.Cu at (329.6, 74.9)
- added REF**: GND Via, Keyboard:GNDVia-wRing, F.Cu at (328.5, 84.6)
- added REF**: GND Via, Keyboard:GNDVia-wRing, F.Cu at (304.5, 85.1)
- added REF**: GND Via, Keyboard:GNDVia-wRing, F.Cu at (273.1, 85.7)
- added REF**: GND Via, Keyboard:GNDVia-wRing, F.Cu at (290.2, 85.7)
- added REF**: GND Via, Keyboard:GNDVia-wRing, F.Cu at (282.6, 66.0)
- added REF**: GND Via, Keyboard:GNDVia-wRing, F.Cu at (229.2, 52.7)
- added REF**: GND Via, Keyboard:GNDVia-wRing, F.Cu at (239.4, 28.6)
- added REF**: GND Via, Keyboard:GNDVia-wRing, F.Cu at (234.3, 31.8)
- added REF**: GND Via, Keyboard:GNDVia-wRing, F.Cu at (245.2, 45.7)
- added REF**: GND Via, Keyboard:GNDVia-wRing, F.Cu at (285.6, 71.3)
- added REF**: GND Via, Keyboard:GNDVia-wRing, F.Cu at (43.3, 38.3)
- added REF**: GND Via, Keyboard:GNDVia-wRing, F.Cu at (44.2, 25.6)
- added REF**: Hole-1mm, Keyboard:Hole-1mm-NPTH, F.Cu at (72.0, 112.0)
- added REF**: GND Via, Keyboard:GNDVia-wRing, F.Cu at (85.3, 23.7)
- added REF**: GND Via, Keyboard:GNDVia-wRing, F.Cu at (106.0, 47.9)
- added REF**: GND Via, Keyboard:GNDVia-wRing, F.Cu at (390.1, 94.3)
- added REF**: GND Via, Keyboard:GNDVia-wRing, F.Cu at (393.6, 86.6)
- added REF**: GND Via, Keyboard:GNDVia-wRing, F.Cu at (392.1, 77.3)
- added REF**: GND Via, Keyboard:GNDVia-wRing, F.Cu at (349.5, 21.0)
- added REF**: GND Via, Keyboard:GNDVia-wRing, F.Cu at (304.7, 22.4)
- added REF**: GND Via, Keyboard:GNDVia-wRing, F.Cu at (277.7, 22.6)
- added REF**: Hole-1mm, Keyboard:Hole-1mm-NPTH, F.Cu at (72.0, 110.0)
- added REF**: GND Via, Keyboard:GNDVia-wRing, F.Cu at (286.2, 22.1)
- added REF**: GND Via, Keyboard:GNDVia-wRing, F.Cu at (259.6, 22.6)
- added REF**: GND Via, Keyboard:GNDVia-wRing, F.Cu at (240.6, 22.8)
- added REF**: GND Via, Keyboard:GNDVia-wRing, F.Cu at (221.1, 22.6)
- added REF**: GND Via, Keyboard:GNDVia-wRing, F.Cu at (182.2, 22.3)
- added REF**: GND Via, Keyboard:GNDVia-wRing, F.Cu at (159.8, 21.5)
- added REF**: GND Via, Keyboard:GNDVia-wRing, F.Cu at (143.0, 21.9)
- added REF**: GND Via, Keyboard:GNDVia-wRing, F.Cu at (398.5, 88.3)
- added REF**: GND Via, Keyboard:GNDVia-wRing, F.Cu at (381.5, 105.3)
- added REF**: Hole-1mm, Keyboard:Hole-1mm-NPTH, F.Cu at (72.0, 108.0)
- added REF**: GND Via, Keyboard:GNDVia-wRing, F.Cu at (377.7, 105.3)
- added REF**: GND Via, Keyboard:GNDVia-wRing, F.Cu at (366.7, 108.1)
- added REF**: GND Via, Keyboard:GNDVia-wRing, F.Cu at (382.9, 85.1)
- added REF**: GND Via, Keyboard:GNDVia-wRing, F.Cu at (386.7, 90.8)
- added REF**: GND Via, Keyboard:GNDVia-wRing, F.Cu at (398.2, 99.7)
- added REF**: GND Via, Keyboard:GNDVia-wRing, F.Cu at (367.3, 72.7)
- added REF**: GND Via, Keyboard:GNDVia-wRing, F.Cu at (373.4, 68.9)
- added REF**: Hole-1mm, Keyboard:Hole-1mm-NPTH, F.Cu at (72.0, 106.0)
- added REF**: GND Via, Keyboard:GNDVia-wRing, F.Cu at (367.0, 68.9)
- added REF**: GND Via, Keyboard:GNDVia-wRing, F.Cu at (340.3, 72.3)
- added REF**: GND Via, Keyboard:GNDVia-wRing, F.Cu at (343.9, 71.0)
- added REF**: GND Via, Keyboard:GNDVia-wRing, F.Cu at (343.9, 67.8)
- added REF**: GND Via, Keyboard:GNDVia-wRing, F.Cu at (346.2, 62.5)
- added REF**: GND Via, Keyboard:GNDVia-wRing, F.Cu at (343.5, 62.5)
- added REF**: GND Via, Keyboard:GNDVia-wRing, F.Cu at (343.5, 57.1)
- added REF**: GND Via, Keyboard:GNDVia-wRing, F.Cu at (346.1, 57.1)
- added REF**: GND Via, Keyboard:GNDVia-wRing, F.Cu at (373.3, 72.5)
- added REF**: GND Via, Keyboard:GNDVia-wRing, F.Cu at (373.6, 60.1)
- added REF**: Hole-1mm, Keyboard:Hole-1mm-NPTH, F.Cu at (72.0, 104.0)
- added REF**: GND Via, Keyboard:GNDVia-wRing, F.Cu at (384.3, 31.3)
- added REF**: GND Via, Keyboard:GNDVia-wRing, F.Cu at (376.8, 21.6)
- added REF**: GND Via, Keyboard:GNDVia-wRing, F.Cu at (360.2, 31.9)
- added REF**: GND Via, Keyboard:GNDVia-wRing, F.Cu at (338.4, 48.2)
- added REF**: GND Via, Keyboard:GNDVia-wRing, F.Cu at (345.2, 40.8)
- added REF**: GND Via, Keyboard:GNDVia-wRing, F.Cu at (295.7, 34.5)
- added REF**: GND Via, Keyboard:GNDVia-wRing, F.Cu at (303.7, 47.7)
- added REF**: Hole-1mm, Keyboard:Hole-1mm-NPTH, F.Cu at (72.0, 102.0)
- added REF**: GND Via, Keyboard:GNDVia-wRing, F.Cu at (319.3, 53.5)
- added REF**: GND Via, Keyboard:GNDVia-wRing, F.Cu at (329.0, 52.9)
- added REF**: GND Via, Keyboard:GNDVia-wRing, F.Cu at (328.9, 46.7)
- added REF**: GND Via, Keyboard:GNDVia-wRing, F.Cu at (323.9, 46.7)
- added REF**: GND Via, Keyboard:GNDVia-wRing, F.Cu at (31.5, 64.3)
- added REF**: Hole-1mm, Keyboard:Hole-1mm-NPTH, F.Cu at (72.0, 98.0)
- added REF**: GND Via, Keyboard:GNDVia-wRing, F.Cu at (31.6, 85.7)
- added REF**: GND Via, Keyboard:GNDVia-wRing, F.Cu at (259.4, 107.8)
- added REF**: GND Via, Keyboard:GNDVia-wRing, F.Cu at (259.4, 98.6)
- added REF**: GND Via, Keyboard:GNDVia-wRing, F.Cu at (248.3, 97.6)
- added REF**: GND Via, Keyboard:GNDVia-wRing, F.Cu at (233.4, 97.8)
- added REF**: GND Via, Keyboard:GNDVia-wRing, F.Cu at (322.0, 74.9)
- added REF**: GND Via, Keyboard:GNDVia-wRing, F.Cu at (322.0, 69.2)
- added REF**: GND Via, Keyboard:GNDVia-wRing, F.Cu at (318.5, 74.9)
- added REF**: GND Via, Keyboard:GNDVia-wRing, F.Cu at (316.7, 79.5)
- added REF**: GND Via, Keyboard:GNDVia-wRing, F.Cu at (128.4, 84.5)
- added REF**: Hole-1mm, Keyboard:Hole-1mm-NPTH, F.Cu at (72.0, 96.0)
- added REF**: GND Via, Keyboard:GNDVia-wRing, F.Cu at (301.0, 66.0)
- added REF**: GND Via, Keyboard:GNDVia-wRing, F.Cu at (285.9, 75.2)
- added REF**: GND Via, Keyboard:GNDVia-wRing, F.Cu at (304.5, 71.1)
- added REF**: GND Via, Keyboard:GNDVia-wRing, F.Cu at (304.3, 79.2)
- added REF**: GND Via, Keyboard:GNDVia-wRing, F.Cu at (301.8, 90.7)
- added REF**: GND Via, Keyboard:GNDVia-wRing, F.Cu at (304.5, 90.7)
- added REF**: GND Via, Keyboard:GNDVia-wRing, F.Cu at (315.0, 85.3)
- added REF**: Hole-1mm, Keyboard:Hole-1mm-NPTH, F.Cu at (72.0, 94.0)
- added REF**: GND Via, Keyboard:GNDVia-wRing, F.Cu at (321.6, 90.4)
- added REF**: GND Via, Keyboard:GNDVia-wRing, F.Cu at (321.7, 82.5)
- added REF**: GND Via, Keyboard:GNDVia-wRing, F.Cu at (314.9, 90.7)
- added REF**: GND Via, Keyboard:GNDVia-wRing, F.Cu at (308.1, 90.7)
- added REF**: GND Via, Keyboard:GNDVia-wRing, F.Cu at (328.9, 110.5)
- added REF**: GND Via, Keyboard:GNDVia-wRing, F.Cu at (316.2, 104.4)
- added REF**: Hole-1mm, Keyboard:Hole-1mm-NPTH, F.Cu at (72.0, 91.0)
- added REF**: GND Via, Keyboard:GNDVia-wRing, F.Cu at (347.1, 67.4)
- added REF**: GND Via, Keyboard:GNDVia-wRing, F.Cu at (354.8, 67.8)
- added REF**: GND Via, Keyboard:GNDVia-wRing, F.Cu at (350.6, 67.5)
- added REF**: GND Via, Keyboard:GNDVia-wRing, F.Cu at (204.1, 62.3)
- added REF**: GND Via, Keyboard:GNDVia-wRing, F.Cu at (202.5, 23.3)
- added REF**: GND Via, Keyboard:GNDVia-wRing, F.Cu at (190.2, 22.7)
- added REF**: GND Via, Keyboard:GNDVia-wRing, F.Cu at (190.3, 30.0)
- added REF**: Hole-1mm, Keyboard:Hole-1mm-NPTH, F.Cu at (72.0, 89.0)
- added REF**: GND Via, Keyboard:GNDVia-wRing, F.Cu at (115.3, 27.5)
- added REF**: GND Via, Keyboard:GNDVia-wRing, F.Cu at (133.7, 27.8)
- added REF**: GND Via, Keyboard:GNDVia-wRing, F.Cu at (171.3, 110.8)
- added REF**: GND Via, Keyboard:GNDVia-wRing, F.Cu at (151.7, 110.9)
- added REF**: GND Via, Keyboard:GNDVia-wRing, F.Cu at (140.9, 105.2)
- added REF**: GND Via, Keyboard:GNDVia-wRing, F.Cu at (171.3, 99.7)
- added REF**: GND Via, Keyboard:GNDVia-wRing, F.Cu at (151.7, 100.0)
- added REF**: Hole-1mm, Keyboard:Hole-1mm-NPTH, F.Cu at (72.0, 87.0)
- added REF**: GND Via, Keyboard:GNDVia-wRing, F.Cu at (136.8, 99.7)
- added REF**: GND Via, Keyboard:GNDVia-wRing, F.Cu at (119.1, 110.1)
- added REF**: GND Via, Keyboard:GNDVia-wRing, F.Cu at (80.2, 90.6)
- added REF**: GND Via, Keyboard:GNDVia-wRing, F.Cu at (85.6, 85.6)
- added REF**: GND Via, Keyboard:GNDVia-wRing, F.Cu at (101.5, 57.3)
- added REF**: GND Via, Keyboard:GNDVia-wRing, F.Cu at (94.3, 57.3)
- added REF**: GND Via, Keyboard:GNDVia-wRing, F.Cu at (114.7, 72.3)
- added REF**: GND Via, Keyboard:GNDVia-wRing, F.Cu at (116.6, 85.7)
- added REF**: Hole-1mm, Keyboard:Hole-1mm-NPTH, F.Cu at (72.0, 85.0)
- added REF**: GND Via, Keyboard:GNDVia-wRing, F.Cu at (113.1, 80.4)
- added REF**: GND Via, Keyboard:GNDVia-wRing, F.Cu at (105.4, 73.0)
- added REF**: GND Via, Keyboard:GNDVia-wRing, F.Cu at (105.7, 79.9)
- added REF**: GND Via, Keyboard:GNDVia-wRing, F.Cu at (108.1, 80.1)
- added REF**: GND Via, Keyboard:GNDVia-wRing, F.Cu at (108.5, 83.4)
- added REF**: GND Via, Keyboard:GNDVia-wRing, F.Cu at (100.3, 82.9)
- added REF**: GND Via, Keyboard:GNDVia-wRing, F.Cu at (97.3, 83.6)
- added REF**: GND Via, Keyboard:GNDVia-wRing, F.Cu at (102.0, 91.1)
- added REF**: GND Via, Keyboard:GNDVia-wRing, F.Cu at (107.6, 92.2)
- added REF**: GND Via, Keyboard:GNDVia-wRing, F.Cu at (140.7, 96.3)
- added REF**: Hole-1mm, Keyboard:Hole-1mm-NPTH, F.Cu at (72.0, 83.0)
- added REF**: GND Via, Keyboard:GNDVia-wRing, F.Cu at (110.2, 103.1)
- added REF**: GND Via, Keyboard:GNDVia-wRing, F.Cu at (99.1, 71.1)
- added REF**: GND Via, Keyboard:GNDVia-wRing, F.Cu at (80.3, 57.4)
- added REF**: GND Via, Keyboard:GNDVia-wRing, F.Cu at (31.5, 25.4)
- added REF**: GND Via, Keyboard:GNDVia-wRing, F.Cu at (80.3, 47.8)
- added REF**: GND Via, Keyboard:GNDVia-wRing, F.Cu at (96.2, 23.3)
- added REF**: GND Via, Keyboard:GNDVia-wRing, F.Cu at (97.7, 103.9)
- added REF**: Hole-1mm, Keyboard:Hole-1mm-NPTH, F.Cu at (72.0, 81.0)
- added REF**: GND Via, Keyboard:GNDVia-wRing, F.Cu at (97.8, 110.0)
- added REF**: GND Via, Keyboard:GNDVia-wRing, F.Cu at (349.9, 42.0)
- added REF**: GND Via, Keyboard:GNDVia-wRing, F.Cu at (361.7, 41.9)
- added REF**: GND Via, Keyboard:GNDVia-wRing, F.Cu at (355.1, 47.2)
- added REF**: GND Via, Keyboard:GNDVia-wRing, F.Cu at (350.5, 47.2)
- added REF**: GND Via, Keyboard:GNDVia-wRing, F.Cu at (361.7, 47.2)
- added REF**: GND Via, Keyboard:GNDVia-wRing, F.Cu at (345.9, 33.5)
- added REF**: GND Via, Keyboard:GNDVia-wRing, F.Cu at (365.3, 23.4)
- added REF**: Hole-1mm, Keyboard:Hole-1mm-NPTH, F.Cu at (72.0, 77.0)
- added REF**: GND Via, Keyboard:GNDVia-wRing, F.Cu at (348.0, 71.9)
- added REF**: GND Via, Keyboard:GNDVia-wRing, F.Cu at (359.7, 75.2)
- added REF**: GND Via, Keyboard:GNDVia-wRing, F.Cu at (348.0, 75.6)
- added REF**: GND Via, Keyboard:GNDVia-wRing, F.Cu at (359.6, 68.0)
- added REF**: GND Via, Keyboard:GNDVia-wRing, F.Cu at (358.0, 63.7)
- added REF**: GND Via, Keyboard:GNDVia-wRing, F.Cu at (286.0, 27.7)
- added REF**: GND Via, Keyboard:GNDVia-wRing, F.Cu at (198.8, 104.1)
- added REF**: GND Via, Keyboard:GNDVia-wRing, F.Cu at (206.2, 111.0)
- added REF**: Hole-1mm, Keyboard:Hole-1mm-NPTH, F.Cu at (72.0, 72.0)
- added REF**: GND Via, Keyboard:GNDVia-wRing, F.Cu at (214.4, 111.0)
- added REF**: GND Via, Keyboard:GNDVia-wRing, F.Cu at (206.0, 100.6)
- added REF**: GND Via, Keyboard:GNDVia-wRing, F.Cu at (363.2, 71.9)
- added REF**: GND Via, Keyboard:GNDVia-wRing, F.Cu at (339.5, 90.1)
- added REF**: GND Via, Keyboard:GNDVia-wRing, F.Cu at (359.7, 90.2)
- added REF**: GND Via, Keyboard:GNDVia-wRing, F.Cu at (360.4, 85.3)
- added REF**: GND Via, Keyboard:GNDVia-wRing, F.Cu at (339.2, 85.1)
- added REF**: GND Via, Keyboard:GNDVia-wRing, F.Cu at (394.3, 97.0)
- added REF**: Hole-1mm, Keyboard:Hole-1mm-NPTH, F.Cu at (72.0, 49.0)
- added REF**: Hole-1mm, Keyboard:Hole-1mm-NPTH, F.Cu at (72.0, 70.0)
- added REF**: GND Via, Keyboard:GNDVia-wRing, F.Cu at (172.1, 85.7)
- added REF**: GND Via, Keyboard:GNDVia-wRing, F.Cu at (229.2, 85.7)
- added REF**: GND Via, Keyboard:GNDVia-wRing, F.Cu at (248.3, 85.1)
- added REF**: GND Via, Keyboard:GNDVia-wRing, F.Cu at (334.0, 47.6)
- added REF**: Hole-1mm, Keyboard:Hole-1mm-NPTH, F.Cu at (72.0, 68.0)
- added REF**: GND Via, Keyboard:GNDVia-wRing, F.Cu at (295.2, 66.0)
- added REF**: Hole-1mm, Keyboard:Hole-1mm-NPTH, F.Cu at (72.0, 66.0)
- added REF**: GND Via, Keyboard:GNDVia-wRing, F.Cu at (48.5, 85.7)
- added REF**: GND Via, Keyboard:GNDVia-wRing, F.Cu at (48.3, 104.8)
- added REF**: GND Via, Keyboard:GNDVia-wRing, F.Cu at (124.8, 103.9)
- added REF**: GND Via, Keyboard:GNDVia-wRing, F.Cu at (105.4, 66.0)
- added REF**: GND Via, Keyboard:GNDVia-wRing, F.Cu at (153.0, 85.7)
- added REF**: Hole-1mm, Keyboard:Hole-1mm-NPTH, F.Cu at (72.0, 64.0)
- added REF**: GND Via, Keyboard:GNDVia-wRing, F.Cu at (288.9, 105.9)
- added REF**: GND Via, Keyboard:GNDVia-wRing, F.Cu at (217.9, 98.3)
- added REF**: GND Via, Keyboard:GNDVia-wRing, F.Cu at (228.1, 110.2)
- added REF**: GND Via, Keyboard:GNDVia-wRing, F.Cu at (307.8, 109.5)
- added REF**: GND Via, Keyboard:GNDVia-wRing, F.Cu at (48.3, 28.6)
- added REF**: Hole-1mm, Keyboard:Hole-1mm-NPTH, F.Cu at (72.0, 62.0)
- added REF**: Hole-1mm, Keyboard:Hole-1mm-NPTH, F.Cu at (72.0, 58.0)
- added REF**: Hole-1mm, Keyboard:Hole-1mm-NPTH, F.Cu at (72.0, 56.0)
- added REF**: Hole-1mm, Keyboard:Hole-1mm-NPTH, F.Cu at (72.0, 53.0)
- added REF**: Hole-1mm, Keyboard:Hole-1mm-NPTH, F.Cu at (72.0, 51.0)
- added REF**: Hole-1mm, Keyboard:Hole-1mm-NPTH, F.Cu at (72.0, 47.0)
- added REF**: Hole-1mm, Keyboard:Hole-1mm-NPTH, F.Cu at (72.0, 45.0)
- added REF**: Hole-1mm, Keyboard:Hole-1mm-NPTH, F.Cu at (72.0, 41.0)
- added REF**: Hole-1mm, Keyboard:Hole-1mm-NPTH, F.Cu at (72.0, 39.0)
- added REF**: Hole-1mm, Keyboard:Hole-1mm-NPTH, F.Cu at (72.0, 37.0)
- added REF**: Hole-1mm, Keyboard:Hole-1mm-NPTH, F.Cu at (72.0, 33.0)
- added REF**: Hole-1mm, Keyboard:Hole-1mm-NPTH, F.Cu at (72.0, 31.0)
- added REF**: Hole-1mm, Keyboard:Hole-1mm-NPTH, F.Cu at (72.0, 29.0)
- added REF**: Hole-1mm, Keyboard:Hole-1mm-NPTH, F.Cu at (72.0, 27.0)
- added REF**: Hole-1mm, Keyboard:Hole-1mm-NPTH, F.Cu at (72.0, 23.0)
- added REF**: Hole-1mm, Keyboard:Hole-1mm-NPTH, F.Cu at (72.0, 21.0)
- added REF**: GND Via, Keyboard:GNDVia-wRing, F.Cu at (193.9, 56.9)
- added REF**: GND Via, Keyboard:GNDVia-wRing, F.Cu at (314.9, 82.4)
- added REF**: GND Via, Keyboard:GNDVia-wRing, F.Cu at (335.2, 76.2)
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Connections:
- C15 pad 1: Net-(C15-Pad1) -> +5V
- D10 pad 1: R1 -> R6
- D11 pad 1: R1 -> R6
- D12 pad 1: R1 -> R6
- D13 pad 1: R1 -> R6
- D14 pad 1: R1 -> R6
- D15 pad 1: R1 -> R6
- D16 pad 1: R1 -> R6
- D17 pad 1: R1 -> R10
- D18 pad 1: R1 -> R10
- D19 pad 1: R2 -> R2/SCK
- D20 pad 1: R2 -> R2/SCK
- D21 pad 1: R2 -> R2/SCK
- D22 pad 1: R2 -> R2/SCK
- D23 pad 1: R2 -> R2/SCK
- D24 pad 1: R2 -> R2/SCK
- D25 pad 1: R2 -> R2/SCK
- D26 pad 1: R2 -> R2/SCK
- D27 pad 1: R2 -> R7
- D28 pad 1: R2 -> R7
- D29 pad 1: R2 -> R7
- D30 pad 1: R2 -> R7
- D31 pad 1: R2 -> R7
- D32 pad 1: R2 -> R7
- D33 pad 1: R2 -> R7
- D34 pad 1: R2 -> R7
- D35 pad 1: R2 -> R10
- D36 pad 1: R2 -> R10
- D37 pad 1: R3 -> R3/MOSI
- D38 pad 1: R3 -> R3/MOSI
- D39 pad 1: R3 -> R3/MOSI
- D40 pad 1: R3 -> R3/MOSI
- D41 pad 1: R3 -> R3/MOSI
- D42 pad 1: R3 -> R3/MOSI
- D43 pad 1: R3 -> R3/MOSI
- D44 pad 1: R3 -> R3/MOSI
- D45 pad 1: R3 -> R8
- D46 pad 1: R3 -> R8
- D47 pad 1: R3 -> R8
- D48 pad 1: R3 -> R8
- D49 pad 1: R3 -> R8
- D50 pad 1: R3 -> R8
- D51 pad 1: R3 -> R8
- D52 pad 1: R4 -> R4/MISO
- D53 pad 1: R4 -> R4/MISO
- D54 pad 1: R4 -> R4/MISO
- D55 pad 1: R4 -> R4/MISO
- D56 pad 1: R4 -> R4/MISO
- D57 pad 1: R4 -> R4/MISO
- D58 pad 1: R4 -> R4/MISO
- D59 pad 1: R4 -> R4/MISO
- D60 pad 1: R4 -> R9
- D61 pad 1: R4 -> R9
- D62 pad 1: R4 -> R9
- D63 pad 1: R4 -> R9
- D64 pad 1: R4 -> R9
- D65 pad 1: R4 -> R9
- D66 pad 1: R4 -> R9
- D75 pad 1: R5 -> R10
- D76 pad 1: Net-(D76-Pad1) -> R10
- D77 pad 1: R5 -> R10
- D78 pad 1: R5 -> R10
- D9 pad 1: R1 -> R6
- R1 pad 1: +5V -> Net-(R1-Pad1)
- R1 pad 2: LED_SDA -> +5V
- R10 pad 1: Net-(R10-Pad1) -> +5V
- R10 pad 2: GND -> LED_SCL
- R11 pad 2: GND -> +5V
- R2 pad 1: +5V -> Net-(R2-Pad1)
- R2 pad 2: LED_SCL -> GND
- R9 pad 1: Net-(R9-Pad1) -> +5V
- R9 pad 2: +5V -> LED_SDA
- SW_Alt_73 pad SW1: C13 -> C7
- SW_B_59 pad SW1: C9 -> C8
- SW_Backspace_16 pad SW1: C16 -> C8
- SW_C_57 pad SW1: C7 -> C6
- SW_Del_35 pad SW1: C17 -> C7
- SW_Enter_51 pad SW1: C15 -> C7
- SW_H_45 pad SW1: C9 -> C1
- SW_I_29 pad SW1: C11 -> C3
- SW_Ins_17 pad SW1: C17 -> C5
- SW_J_46 pad SW1: C10 -> C2
- SW_K_47 pad SW1: C11 -> C3
- SW_L_48 pad SW1: C12 -> C4
- SW_M_61 pad SW1: C11 -> C2
- SW_Menu_75 pad SW1: C15 -> C1
- SW_N_60 pad SW1: C10 -> C1
- SW_O_30 pad SW1: C12 -> C4
- SW_P_31 pad SW1: C13 -> C5
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Routing:
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Other:
- board size 367.8 x 92.5 mm -> 370.5 x 94.4 mm
- net class Default: trace_width 0.3048 -> 0.381; via_dia 0.6858 -> 0.6096; via_drill 0.3302 -> 0.3048
- net class USB removed
- net class backlight removed
- net class matrix removed
- net class power removed
- net class underglow removed
- rule trace_min: 0.1524 -> 0.254
- rule via_min_drill: 0.3302 -> 0.3048
- rule via_min_size: 0.6858 -> 0.6096
- board text added: "CENTER"
- board text added: "Single Quote"
- board text removed: "LFK78 RevC"
- board text removed: "LFK78 RevC - ISO/ANSI"
- board text removed: "Quote"
- board text removed: "https://github.com/mechkeys/mechkeys"

Commit message: Added reversible mini layout
Parts:
- removed the CHERRY at (338.1, 28.6)
- removed the REF** at (72.0, 112.0)
- removed the REF** at (349.5, 21.0)
- removed the REF** at (72.0, 110.0)
- removed the REF** at (398.5, 88.3)
- removed the REF** at (72.0, 108.0)
- removed the REF** at (398.2, 99.7)
- removed the REF** at (72.0, 106.0)
- removed the REF** at (72.0, 104.0)
- removed the REF** at (72.0, 102.0)
- removed the REF** at (31.5, 64.3)
- removed the REF** at (72.0, 98.0)
- removed the REF** at (259.4, 98.6)
- removed the REF** at (248.3, 97.6)
- removed the REF** at (233.4, 97.8)
- removed the REF** at (72.0, 96.0)
- removed the REF** at (72.0, 94.0)
- removed the REF** at (72.0, 91.0)
- removed the REF** at (72.0, 89.0)
- removed the REF** at (72.0, 87.0)
- removed the REF** at (72.0, 85.0)
- removed the REF** at (72.0, 83.0)
- removed the REF** at (72.0, 81.0)
- removed the REF** at (72.0, 77.0)
- removed the REF** at (198.8, 104.1)
- removed the REF** at (72.0, 72.0)
- removed the REF** at (206.0, 100.6)
- removed the REF** at (72.0, 49.0)
- removed the REF** at (72.0, 70.0)
- removed the REF** at (72.0, 68.0)
- removed the REF** at (72.0, 66.0)
- removed the REF** at (72.0, 64.0)
- removed the REF** at (307.8, 109.5)
- removed the REF** at (72.0, 62.0)
- removed the REF** at (72.0, 58.0)
- removed the REF** at (72.0, 56.0)
- removed the REF** at (72.0, 53.0)
- removed the REF** at (72.0, 51.0)
- removed the REF** at (72.0, 47.0)
- removed the REF** at (72.0, 45.0)
- removed the REF** at (72.0, 41.0)
- removed the REF** at (72.0, 39.0)
- removed the REF** at (72.0, 37.0)
- removed the REF** at (72.0, 33.0)
- removed the REF** at (72.0, 31.0)
- removed the REF** at (72.0, 29.0)
- removed the REF** at (72.0, 27.0)
- removed the REF** at (72.0, 23.0)
- removed the REF** at (72.0, 21.0)
- removed the REF** at (73.5, 90.0)
- removed the REF** at (73.5, 84.0)
- removed the REF** at (73.5, 71.0)
- removed the REF** at (73.5, 65.0)
- removed the REF** at (73.5, 57.0)
- removed the REF** at (73.5, 48.0)
- removed the REF** at (193.0, 97.3)
- added REF**: GND Via, Keyboard:GNDVia-wRing, F.Cu at (191.0, 96.2)
- added REF**: GND Via, Keyboard:GNDVia-wRing, F.Cu at (171.3, 96.2)
- added REF**: GND Via, Keyboard:GNDVia-wRing, F.Cu at (228.0, 99.5)
- added REF**: GND Via, Keyboard:GNDVia-wRing, F.Cu at (254.0, 100.5)
- added REF**: GND Via, Keyboard:GNDVia-wRing, F.Cu at (102.5, 21.5)
- added REF**: GND Via, Keyboard:GNDVia-wRing, F.Cu at (396.0, 34.0)
- added REF**: GND Via, Keyboard:GNDVia-wRing, F.Cu at (117.5, 89.3)
- added REF**: GND Via, Keyboard:GNDVia-wRing, F.Cu at (99.3, 80.6)
- moved REF** 25.9 mm to (122.0, 21.5)
- moved REF** 17.5 mm to (35.0, 94.0)
- moved REF** 17.4 mm to (388.5, 56.0)
- moved REF** 15.6 mm to (34.5, 57.5)
- moved REF** 6.94 mm to (396.0, 38.5)
- moved REF** 5.63 mm to (254.0, 109.5)
- moved REF** 5.24 mm to (78.7, 38.1)
- moved REF** 4.08 mm to (77.5, 106.0)
- moved REF** 3.43 mm to (76.8, 97.8)
- moved REF** 3.28 mm to (217.5, 110.0)
- moved REF** 3.27 mm to (33.5, 83.0)
- moved REF** 3.18 mm to (304.0, 109.8)
- moved REF** 3.09 mm to (396.0, 63.0)
- moved REF** 2.77 mm to (395.0, 22.0)
- moved REF** 2.51 mm to (34.0, 25.5)
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Routing:
- net AUDIO: track 180.5 -> 172.3 mm
- net R_CB1: track 322.9 -> 317.6 mm
- net C1: track 524.1 -> 521.1 mm
- net C4: track 496.9 -> 495.3 mm
Other:
- board size 370.5 x 94.4 mm -> 367.8 x 92.5 mm
- board text added: "LFK78 RevA"
- board text added: "Quote"
- board text added: "https://github.com/mechkeys/mechkeys"
- board text removed: "Single Quote"
