File: LFK78/LFK78.sch (KiCad schematic (older format))
At the start: 180 parts, among them J1 USB_OTG, SW1 SW_RST, U2 AT90USB1286, X1 16Mhz, X2 PiezoelectricCrystal-TwoElect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

Commit message: Rollback LFK78 to the actual oder made in Oct
Parts:
- removed D79: D, Diodes_ThroughHole:Diode_DO-35_SOD27_Horizontal_RM10, symbol D
- removed SW_ISO_SLASH_79: MX_LED, symbol MX_LED
- removed U2: AT90USB1286, Housings_QFP:TQFP-64_14x14mm_Pitch0.8mm, symbol AT90USB1286
- added C1, C14: 1µF, Capacitors_SMD:C_0805, symbol C
- added C15, C16, C2, C3: 0.1µF, Capacitors_SMD:C_0805, symbol C_Small
- added R1, R11: 10KΩ, Resistors_SMD:R_0805, symbol R
- added R10, R9: 4.7KΩ, Resistors_SMD:R_0805, symbol R
- added R13, R2: 20KΩ, Resistors_SMD:R_0805, symbol R
- added RGB1, RGB10, RGB11, RGB12, RGB13, RGB14, RGB15, RGB16, RGB17, RGB18, RGB19, RGB2, RGB20, RGB21, RGB22, RGB23, RGB24, RGB25, RGB26, RGB27, RGB28, RGB29, RGB3, RGB30, RGB31, RGB32, RGB4, RGB5, RGB6, RGB7, RGB8, RGB9: Led_RGB_CA, symbol Led_RGB_CA
- added unit 2 of SW_A_40
- added unit 2 of SW_Alt_71
- added unit 2 of SW_Alt_73
- added unit 2 of SW_B_59
- added unit 2 of SW_Backspace_16
- added unit 2 of SW_C_57
- added unit 2 of SW_Caps_39
- added unit 2 of SW_Ctrl_69
- added unit 2 of SW_D_42
- added unit 2 of SW_Del_35
- added unit 2 of SW_E_24
- added unit 2 of SW_Enter_51
- added unit 2 of SW_F10_68
- added unit 2 of SW_F1_1
- added unit 2 of SW_F2_2
- added unit 2 of SW_F3_19
- added unit 2 of SW_F4_20
- added unit 2 of SW_F5_37
- added unit 2 of SW_F6_38
- added unit 2 of SW_F7_52
- added unit 2 of SW_F8_53
- added unit 2 of SW_F9_67
- added unit 2 of SW_F_43
- added unit 2 of SW_G_44
- added unit 2 of SW_H_45
- added unit 2 of SW_I_29
- added unit 2 of SW_Ins_17
- added unit 2 of SW_J_46
- added unit 2 of SW_K_47
- added unit 2 of SW_L_48
- added unit 2 of SW_M_61
- added unit 2 of SW_Menu_75
- added unit 2 of SW_N_60
- added unit 2 of SW_O_30
- added unit 2 of SW_P_31
- added unit 2 of SW_PgDn_36
- added unit 2 of SW_PgUp_18
- added unit 2 of SW_Q_22
- added unit 2 of SW_R_25
- added unit 2 of SW_S_41
- added unit 2 of SW_Shift_54
- added unit 2 of SW_Shift_65
- added unit 2 of SW_T_26
- added unit 2 of SW_Tab_21
- added unit 2 of SW_U_28
- added unit 2 of SW_V_58
- added unit 2 of SW_W_23
- added unit 2 of SW_Win_70
- added unit 2 of SW_Win_74
- added unit 2 of SW_X10Y1_9
- added unit 2 of SW_X11Y1_10
- added unit 2 of SW_X12Y1_11
- added unit 2 of SW_X13Y1_12
- added unit 2 of SW_X13Y4_62
- added unit 2 of SW_X14Y1_13
- added unit 2 of SW_X14Y4_63
- added unit 2 of SW_X15Y1_14
- added unit 2 of SW_X15Y2_32
- added unit 2 of SW_X15Y3_49
- added unit 2 of SW_X15Y4_64
- added unit 2 of SW_X16Y1_15
- added unit 2 of SW_X16Y2_33
- added unit 2 of SW_X16Y3_50
- added unit 2 of SW_X17Y2_34
- added unit 2 of SW_X18Y5_76
- added unit 2 of SW_X19Y4_66
- added unit 2 of SW_X19Y5_77
- added unit 2 of SW_X20Y5_78
- added unit 2 of SW_X4Y1_3
- added unit 2 of SW_X5Y1_4
- added unit 2 of SW_X6Y1_5
- added unit 2 of SW_X7Y1_6
- added unit 2 of SW_X8Y1_7
- added unit 2 of SW_X8Y5_72
- added unit 2 of SW_X9Y1_8
- added unit 2 of SW_X_56
- added unit 2 of SW_Y_27
- added unit 2 of SW_Z_55
- added U1: ATMEGA32U4RC-A, Housings_QFP:TQFP-44_10x10mm_Pitch0.8mm, symbol ATMEGA32U4RC-A
- added U2, U3: IS31FL3731, Housings_SSOP:SSOP-28_5.3x10.2mm_Pitch0.65mm, symbol IS31FL3731
Connections:
- net labels added: L_CA1, L_CA2, L_CA3, L_CA4, L_CA5, L_CA6, L_CA7, L_CA8, L_CA9, L_CB1, L_CB2, L_CB3, L_CB4, L_CB5, L_CB6, L_CB7, L_CB8, L_CB9, R10, R2/SCK, R3/MOSI, R4/MISO, R6, R7, R8, R9, R_CA1, R_CA2, R_CA3, R_CA4, R_CA5, R_CA6, R_CA7, R_CA8, R_CA9, R_CB1, R_CB2, R_CB3, R_CB4, R_CB5, R_CB6, R_CB7, R_CB8, R_CB9
- net labels removed: C10, C11, C12, C13, C14, C15, C16, C17, C18, C9, MISO, MOSI, R2, R3, R4, SCK
- wire segments 188 -> 566
Other:
- moved on the sheet: C10, C11, C12, C4, C5, C6, C7, C8, C9, D54, D65, D66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

Commit message: LFK78 RevC addedd
Parts:
- removed C1, C14: 1µF, Capacitors_SMD:C_0805, symbol C
- removed C15, C16, C2, C3: 0.1µF, Capacitors_SMD:C_0805, symbol C_Small
- removed R1, R11: 10KΩ, Resistors_SMD:R_0805, symbol R
- removed R10, R9: 4.7KΩ, Resistors_SMD:R_0805, symbol R
- removed R13, R2: 20KΩ, Resistors_SMD:R_0805, symbol R
- removed RGB1, RGB10, RGB11, RGB12, RGB13, RGB14, RGB15, RGB16, RGB17, RGB18, RGB19, RGB2, RGB20, RGB21, RGB22, RGB23, RGB24, RGB25, RGB26, RGB27, RGB28, RGB29, RGB3, RGB30, RGB31, RGB32, RGB4, RGB5, RGB6, RGB7, RGB8, RGB9: Led_RGB_CA, symbol Led_RGB_CA
- removed unit 2 of SW_A_40
- removed unit 2 of SW_Alt_71
- removed unit 2 of SW_Alt_73
- removed unit 2 of SW_B_59
- removed unit 2 of SW_Backspace_16
- removed unit 2 of SW_C_57
- removed unit 2 of SW_Caps_39
- removed unit 2 of SW_Ctrl_69
- removed unit 2 of SW_D_42
- removed unit 2 of SW_Del_35
- removed unit 2 of SW_E_24
- removed unit 2 of SW_Enter_51
- removed unit 2 of SW_F10_68
- removed unit 2 of SW_F1_1
- removed unit 2 of SW_F2_2
- removed unit 2 of SW_F3_19
- removed unit 2 of SW_F4_20
- removed unit 2 of SW_F5_37
- removed unit 2 of SW_F6_38
- removed unit 2 of SW_F7_52
- removed unit 2 of SW_F8_53
- removed unit 2 of SW_F9_67
- removed unit 2 of SW_F_43
- removed unit 2 of SW_G_44
- removed unit 2 of SW_H_45
- removed unit 2 of SW_I_29
- removed unit 2 of SW_Ins_17
- removed unit 2 of SW_J_46
- removed unit 2 of SW_K_47
- removed unit 2 of SW_L_48
- removed unit 2 of SW_M_61
- removed unit 2 of SW_Menu_75
- removed unit 2 of SW_N_60
- removed unit 2 of SW_O_30
- removed unit 2 of SW_P_31
- removed unit 2 of SW_PgDn_36
- removed unit 2 of SW_PgUp_18
- removed unit 2 of SW_Q_22
- removed unit 2 of SW_R_25
- removed unit 2 of SW_S_41
- removed unit 2 of SW_Shift_54
- removed unit 2 of SW_Shift_65
- removed unit 2 of SW_T_26
- removed unit 2 of SW_Tab_21
- removed unit 2 of SW_U_28
- removed unit 2 of SW_V_58
- removed unit 2 of SW_W_23
- removed unit 2 of SW_Win_70
- removed unit 2 of SW_Win_74
- removed unit 2 of SW_X10Y1_9
- removed unit 2 of SW_X11Y1_10
- removed unit 2 of SW_X12Y1_11
- removed unit 2 of SW_X13Y1_12
- removed unit 2 of SW_X13Y4_62
- removed unit 2 of SW_X14Y1_13
- removed unit 2 of SW_X14Y4_63
- removed unit 2 of SW_X15Y1_14
- removed unit 2 of SW_X15Y2_32
- removed unit 2 of SW_X15Y3_49
- removed unit 2 of SW_X15Y4_64
- removed unit 2 of SW_X16Y1_15
- removed unit 2 of SW_X16Y2_33
- removed unit 2 of SW_X16Y3_50
- removed unit 2 of SW_X17Y2_34
- removed unit 2 of SW_X18Y5_76
- removed unit 2 of SW_X19Y4_66
- removed unit 2 of SW_X19Y5_77
- removed unit 2 of SW_X20Y5_78
- removed unit 2 of SW_X4Y1_3
- removed unit 2 of SW_X5Y1_4
- removed unit 2 of SW_X6Y1_5
- removed unit 2 of SW_X7Y1_6
- removed unit 2 of SW_X8Y1_7
- removed unit 2 of SW_X8Y5_72
- removed unit 2 of SW_X9Y1_8
- removed unit 2 of SW_X_56
- removed unit 2 of SW_Y_27
- removed unit 2 of SW_Z_55
- removed U1: ATMEGA32U4RC-A, Housings_QFP:TQFP-44_10x10mm_Pitch0.8mm, symbol ATMEGA32U4RC-A
- removed U2, U3: IS31FL3731, Housings_SSOP:SSOP-28_5.3x10.2mm_Pitch0.65mm, symbol IS31FL3731
- added D79: D, Diodes_ThroughHole:Diode_DO-35_SOD27_Horizontal_RM10, symbol D
- added SW_ISO_SLASH_79: MX_LED, symbol MX_LED
- added U2: AT90USB1286, Housings_QFP:TQFP-64_14x14mm_Pitch0.8mm, symbol AT90USB1286
Connections:
- net labels added: C10, C11, C12, C13, C14, C15, C16, C17, C18, C9, MISO, MOSI, R2, R3, R4, SCK
- net labels removed: L_CA1, L_CA2, L_CA3, L_CA4, L_CA5, L_CA6, L_CA7, L_CA8, L_CA9, L_CB1, L_CB2, L_CB3, L_CB4, L_CB5, L_CB6, L_CB7, L_CB8, L_CB9, R10, R2/SCK, R3/MOSI, R4/MISO, R6, R7, R8, R9, R_CA1, R_CA2, R_CA3, R_CA4, R_CA5, R_CA6, R_CA7, R_CA8, R_CA9, R_CB1, R_CB2, R_CB3, R_CB4, R_CB5, R_CB6, R_CB7, R_CB8, R_CB9
- wire segments 566 -> 188
Other:
- moved on the sheet: C10, C11, C12, C4, C5, C6, C7, C8, C9, D54, D65, D66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
