File: lfk_revc/lfk_revc.kicad_pcb (KiCad board)
At the start: 2 copper layers, 371.5 x 95.2 mm, 241 parts, among them P1 USB_B, P2 CONN_02X03, SW1 SW_PUSH, U1 AT90USB1286, U2 IS31FL3731, U3 IS31FL3731, Y1 16Mhz

Commit message: revC board completed with USB and mounting holes verified for VA68M case.
Parts:
- removed the RGB13 at (239.1, 123.3)
- removed the RGB14 at (211.1, 154.5)
- removed RGB15, RGB23, RGB26, RGB27, RGB29: Led_RGB_CA, Keyboard:SMP4-RGB
- removed the RGB33 at (267.8, 144.1)
- removed the RGB8 at (201.6, 146.9)
- removed SW_82, SW_85: MX_LED, MXALPS
- removed SW_86: MX_LED, Keyboard:MXALPS_REVERSE_LED
- added P3: CONN_02X05, Pin_Headers:Pin_Header_Straight_2x05, B.Cu at (349.2, 87.6)
- added P4: CONN_01X03, Pin_Headers:Pin_Header_Straight_1x03, B.Cu at (381.0, 83.2)
- added REF**: GND Via, Keyboard:GNDVia-wRing, F.Cu at (354.5, 59.2)
- added REF**: GND Via, Keyboard:GNDVia-wRing, F.Cu at (64.4, 68.7)
- added REF**: GND Via, Keyboard:GNDVia-wRing, F.Cu at (77.2, 87.4)
- added REF**: GND Via, Keyboard:GNDVia-wRing, F.Cu at (78.5, 80.0)
- added REF**: GND Via, Keyboard:GNDVia-wRing, F.Cu at (78.5, 70.5)
- added REF**: GND Via, Keyboard:GNDVia-wRing, F.Cu at (78.8, 60.6)
- added REF**: GND Via, Keyboard:GNDVia-wRing, F.Cu at (78.8, 49.7)
- added REF**: GND Via, Keyboard:GNDVia-wRing, F.Cu at (174.6, 45.7)
- added REF**: GND Via, Keyboard:GNDVia-wRing, F.Cu at (172.7, 57.8)
- added REF**: GND Via, Keyboard:GNDVia-wRing, F.Cu at (163.2, 57.8)
- added REF**: GND Via, Keyboard:GNDVia-wRing, F.Cu at (124.5, 57.1)
- added REF**: GND Via, Keyboard:GNDVia-wRing, F.Cu at (373.5, 64.6)
- added REF**: GND Via, Keyboard:GNDVia-wRing, F.Cu at (78.7, 41.3)
- added REF**: GND Via, Keyboard:GNDVia-wRing, F.Cu at (34.3, 44.5)
- added REF**: GND Via, Keyboard:GNDVia-wRing, F.Cu at (33.7, 24.8)
- added REF**: GND Via, Keyboard:GNDVia-wRing, F.Cu at (45.7, 26.7)
- added REF**: GND Via, Keyboard:GNDVia-wRing, F.Cu at (57.1, 110.5)
- added REF**: GND Via, Keyboard:GNDVia-wRing, F.Cu at (34.3, 102.9)
- added REF**: GND Via, Keyboard:GNDVia-wRing, F.Cu at (53.3, 94.0)
- added REF**: GND Via, Keyboard:GNDVia-wRing, F.Cu at (53.3, 79.4)
- added REF**: GND Via, Keyboard:GNDVia-wRing, F.Cu at (53.3, 57.1)
- added REF**: GND Via, Keyboard:GNDVia-wRing, F.Cu at (280.0, 106.7)
- added REF**: GND Via, Keyboard:GNDVia-wRing, F.Cu at (374.3, 74.9)
- added REF**: GND Via, Keyboard:GNDVia-wRing, F.Cu at (311.1, 87.0)
- added REF**: GND Via, Keyboard:GNDVia-wRing, F.Cu at (323.9, 73.0)
- added REF**: GND Via, Keyboard:GNDVia-wRing, F.Cu at (343.5, 66.7)
- added REF**: GND Via, Keyboard:GNDVia-wRing, F.Cu at (343.5, 71.8)
- added REF**: GND Via, Keyboard:GNDVia-wRing, F.Cu at (361.3, 80.6)
- added REF**: GND Via, Keyboard:GNDVia-wRing, F.Cu at (362.6, 50.2)
- added REF**: GND Via, Keyboard:GNDVia-wRing, F.Cu at (357.5, 50.2)
- added REF**: GND Via, Keyboard:GNDVia-wRing, F.Cu at (365.8, 37.5)
- added REF**: GND Via, Keyboard:GNDVia-wRing, F.Cu at (342.9, 25.4)
- added REF**: GND Via, Keyboard:GNDVia-wRing, F.Cu at (377.8, 26.0)
- added REF**: GND Via, Keyboard:GNDVia-wRing, F.Cu at (361.2, 77.1)
- added REF**: GND Via, Keyboard:GNDVia-wRing, F.Cu at (395.6, 36.2)
- added REF**: GND Via, Keyboard:GNDVia-wRing, F.Cu at (390.5, 66.7)
- added REF**: GND Via, Keyboard:GNDVia-wRing, F.Cu at (381.0, 63.5)
- added REF**: GND Via, Keyboard:GNDVia-wRing, F.Cu at (381.0, 61.0)
- added REF**: GND Via, Keyboard:GNDVia-wRing, F.Cu at (379.7, 57.8)
- added REF**: GND Via, Keyboard:GNDVia-wRing, F.Cu at (380.4, 71.8)
- added REF**: GND Via, Keyboard:GNDVia-wRing, F.Cu at (373.4, 69.8)
- added REF**: GND Via, Keyboard:GNDVia-wRing, F.Cu at (365.8, 63.5)
- added REF**: GND Via, Keyboard:GNDVia-wRing, F.Cu at (332.7, 57.8)
- added REF**: GND Via, Keyboard:GNDVia-wRing, F.Cu at (299.7, 23.5)
- added REF**: GND Via, Keyboard:GNDVia-wRing, F.Cu at (354.1, 74.5)
- added REF**: GND Via, Keyboard:GNDVia-wRing, F.Cu at (325.8, 29.8)
- added REF**: GND Via, Keyboard:GNDVia-wRing, F.Cu at (306.7, 57.1)
- added REF**: GND Via, Keyboard:GNDVia-wRing, F.Cu at (258.4, 57.8)
- added REF**: GND Via, Keyboard:GNDVia-wRing, F.Cu at (182.9, 57.8)
- added REF**: GND Via, Keyboard:GNDVia-wRing, F.Cu at (242.6, 23.5)
- added REF**: GND Via, Keyboard:GNDVia-wRing, F.Cu at (204.5, 24.8)
- added REF**: GND Via, Keyboard:GNDVia-wRing, F.Cu at (153.0, 23.5)
- added REF**: GND Via, Keyboard:GNDVia-wRing, F.Cu at (114.9, 23.5)
- added REF**: GND Via, Keyboard:GNDVia-wRing, F.Cu at (75.6, 23.5)
- added REF**: GND Via, Keyboard:GNDVia-wRing, F.Cu at (190.5, 106.0)
- added REF**: GND Via, Keyboard:GNDVia-wRing, F.Cu at (89.7, 103.0)
- added REF**: GND Via, Keyboard:GNDVia-wRing, F.Cu at (153.0, 106.7)
- added REF**: GND Via, Keyboard:GNDVia-wRing, F.Cu at (96.5, 106.7)
- added REF**: GND Via, Keyboard:GNDVia-wRing, F.Cu at (114.9, 85.7)
- added REF**: GND Via, Keyboard:GNDVia-wRing, F.Cu at (133.3, 85.7)
- added REF**: GND Via, Keyboard:GNDVia-wRing, F.Cu at (153.0, 85.7)
- added REF**: GND Via, Keyboard:GNDVia-wRing, F.Cu at (171.4, 85.7)
- added REF**: GND Via, Keyboard:GNDVia-wRing, F.Cu at (190.5, 85.7)
- added REF**: GND Via, Keyboard:GNDVia-wRing, F.Cu at (209.6, 85.7)
- added REF**: GND Via, Keyboard:GNDVia-wRing, F.Cu at (228.6, 85.7)
- added REF**: GND Via, Keyboard:GNDVia-wRing, F.Cu at (241.3, 83.2)
- added REF**: GND Via, Keyboard:GNDVia-wRing, F.Cu at (77.2, 109.6)
- added REF**: GND Via, Keyboard:GNDVia-wRing, F.Cu at (280.0, 83.2)
- added REF**: GND Via, Keyboard:GNDVia-wRing, F.Cu at (285.8, 87.1)
- added REF**: GND Via, Keyboard:GNDVia-wRing, F.Cu at (266.7, 87.1)
- added REF**: GND Via, Keyboard:GNDVia-wRing, F.Cu at (266.7, 109.7)
- added REF**: GND Via, Keyboard:GNDVia-wRing, F.Cu at (222.0, 109.3)
- added REF**: GND Via, Keyboard:GNDVia-wRing, F.Cu at (247.7, 99.2)
- added REF**: GND Via, Keyboard:GNDVia-wRing, F.Cu at (235.6, 107.3)
- added REF**: GND Via, Keyboard:GNDVia-wRing, F.Cu at (242.9, 95.9)
- added REF**: GND Via, Keyboard:GNDVia-wRing, F.Cu at (391.2, 72.6)
- added REF**: GND Via, Keyboard:GNDVia-wRing, F.Cu at (63.8, 89.8)
- added REF**: GND Via, Keyboard:GNDVia-wRing, F.Cu at (357.6, 62.9)
- added REF**: GND Via, Keyboard:GNDVia-wRing, F.Cu at (64.4, 41.3)
- added RGB13: Led_RGB_CA, Keyboard:SMP4-RGB, B.Cu at (80.6, 38.1)
- added RGB13: Led_RGB_CA, Keyboard:SMP4-RGB, B.Cu at (38.1, 38.1)
- added RGB14: Led_RGB_CA, Keyboard:SMP4-RGB, B.Cu at (80.6, 57.1)
- added RGB14: Led_RGB_CA, Keyboard:SMP4-RGB, B.Cu at (38.1, 57.1)
- added RGB8: Led_RGB_CA, Keyboard:SMP4-RGB, B.Cu at (80.6, 76.2)
- added RGB8: Led_RGB_CA, Keyboard:SMP4-RGB, B.Cu at (38.1, 76.2)
- added STA: Stabilizer, Keyboard:CHERRY_PCB_200_STABILIZER_OUTLINE, F.Cu at (338.1, 28.6)
- added STA: Stabilizer, Keyboard:CHERRY_PCB_200_STABILIZER_OUTLINE, F.Cu at (331.7, 126.6)
- added SW_40: MX_LED, MXALPS, F.Cu at (83.3, 66.7)
- C10, C11, C13, C14, C15, C3, C6, C7, C8, C9, R1, R11, R12, R13, R14, R2, R3, RGB1, RGB10, RGB11, RGB12, RGB16, RGB17, RGB18, RGB19, RGB2, RGB20, RGB21, RGB22, RGB24, RGB25, RGB28, RGB3, RGB30, RGB31, RGB32, RGB4, RGB5, RGB6, RGB7, RGB9: moved to B.Cu
- C12: footprint Capacitors_SMD:C_0805 -> Capacitors_SMD:C_0805_HandSoldering
- P2: footprint Pin_Headers:Pin_Header_Angled_2x03 -> Pin_Headers:Pin_Header_Straight_2x03; moved to B.Cu
- R6: value 4.7kΩ -> 150; moved to B.Cu
- R7, R8: value 4.7kΩ -> 120; moved to B.Cu
- moved C3 206.4 mm to (364.5, 56.3), turned to 180 degrees
- moved RGB12 201.1 mm to (48.3, 30.0), turned to 270 degrees
- moved C8 196.8 mm to (375.3, 58.5)
- moved C9 191.3 mm to (375.3, 60.7), turned to 180 degrees
- moved P2 189.4 mm to (356.9, 31.0), turned to 270 degrees
- moved RGB28 188.1 mm to (380.5, 30.0), turned to 270 degrees
- moved R1 183.0 mm to (390.5, 59.7)
- moved C6 182.5 mm to (350.6, 70.9), turned to 180 degrees
- moved C7 179.3 mm to (350.6, 68.7)
- moved RGB22 178.6 mm to (390.5, 76.2), turned to 270 degrees
- moved RGB7 177.2 mm to (38.1, 95.2), turned to 270 degrees
- moved RGB25 176.1 mm to (390.5, 38.1), turned to 270 degrees
- moved RGB24 174.3 mm to (390.5, 57.1), turned to 270 degrees
- moved RGB11 169.1 mm to (90.4, 30.0), turned to 270 degrees
- moved R6 161.0 mm to (389.1, 81.5), turned to 180 degrees
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Connections:
- D17 pad 1: Net-(D17-Pad1) -> R1
- D18 pad 1: Net-(D18-Pad1) -> R1
- D36 pad 1: Net-(D36-Pad1) -> R2
- D37 pad 1: Net-(D37-Pad1) -> R2
- D70 pad 1: Net-(D70-Pad1) -> R4
- D89 pad 1: Net-(D89-Pad1) -> R5
- D90 pad 1: Net-(D90-Pad1) -> R5
- D91 pad 1: Net-(D91-Pad1) -> R5
- P1 pad 6: (no net) -> GND
- RGB1 pad 1: R_CA1 -> R_CA2
- RGB2 pad 1: R_CA2 -> R_CA3
- RGB3 pad 1: R_CA3 -> R_CA4
- RGB4 pad 1: R_CA4 -> R_CA5
- RGB5 pad 1: Net-(RGB5-Pad1) -> R_CA6
- RGB6 pad 1: R_CA6 -> R_CA7
- RGB7 pad 1: Net-(RGB7-Pad1) -> R_CA8
- SW_17 pad SW1: Net-(SW_17-PadSW1) -> C17
- SW_18 pad SW1: Net-(SW_18-PadSW1) -> C18
- SW_36 pad SW1: Net-(SW_36-PadSW1) -> C17
- SW_37 pad SW1: Net-(SW_37-PadSW1) -> C18
- SW_70 pad SW1: Net-(SW_70-PadSW1) -> C17
- SW_89 pad SW1: Net-(SW_89-PadSW1) -> C16
- SW_90 pad SW1: Net-(SW_90-PadSW1) -> C17
- SW_91 pad SW1: Net-(SW_91-PadSW1) -> C18
- U1 pad 35: Net-(U1-Pad35) -> C15
- U1 pad 36: Net-(U1-Pad36) -> C16
- U1 pad 37: Net-(U1-Pad37) -> C17
- U1 pad 38: Net-(U1-Pad38) -> C18
- U1 pad 54: C18 -> TDI
- U1 pad 55: C17 -> TDO
- U1 pad 56: C16 -> TMS
- U1 pad 57: C15 -> TCK
- Y1 pad 3: (no net) -> GND
Routing:
- net R_CA7: track 0.00 -> 564.7 mm, vias 0 -> 13
- net R_CA8: track 0.00 -> 530.3 mm, vias 0 -> 8
- net +5V: track 0.00 -> 436.8 mm, vias 0 -> 12
- net R_CA9: track 0.00 -> 432.4 mm, vias 0 -> 8
- net R_CA1: track 0.00 -> 371.9 mm, vias 0 -> 8
- net R_CA6: track 0.00 -> 367.1 mm, vias 0 -> 7
- net R_CA3: track 0.00 -> 352.1 mm, vias 0 -> 10
- net R_CB6: track 0.00 -> 334.2 mm, vias 0 -> 4
- net R_CA5: track 0.00 -> 331.1 mm, vias 0 -> 7
- net C1: track 76.2 -> 392.7 mm, vias 0 -> 1
- net R_CB7: track 0.00 -> 312.7 mm, vias 0 -> 8
- net R_CB9: track 0.00 -> 304.4 mm, vias 0 -> 8
- net C2: track 76.2 -> 372.7 mm, vias 0 -> 1
- net R_CB8: track 0.00 -> 279.4 mm, vias 0 -> 4
- net R_CA4: track 0.00 -> 276.1 mm, vias 0 -> 6
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Other:
- board size 371.5 x 95.2 mm -> 367.8 x 93.2 mm
- net class Default: clearance 0.2032 -> 0.19685
- net class USB added: clearance 0.2032, trace_width 0.2032, via_dia 0.6858, via_drill 0.3302
- net class backlight: clearance 0.2032 -> 0.19685
- rule pad_to_mask_clearance: 0.2 -> 0.04
- rule trace_clearance: 0.2032 -> 0.19685
- board text added: "'"
- board text added: "+"
- board text added: "+5v"
- board text added: "-"
- board text added: "/"
- board text added: "0"
- board text added: "1"
- board text added: "2"
- board text added: "3"
- board text added: "4"
- board text added: "5"
- board text added: "6"
- board text added: "7"
- board text added: "8"
- board text added: "9"
- board text added: ";"
- board text added: "A"
- board text added: "B"
- board text added: "Backspace"
- board text added: "C"
- board text added: "Caps"
- board text added: "Comma"
- board text added: "D"
- board text added: "Delete"
- board text added: "Down"
- board text added: "E"
- board text added: "Enter"
- board text added: "Escape"
- board text added: "F"
- board text added: "F1"
- board text added: "F10"
- board text added: "F2"
- board text added: "F3"
- board text added: "F4"
- board text added: "F5"
- board text added: "F6"
- board text added: "F7"
- board text added: "F8"
- board text added: "F9"
- board text added: "G"
- board text added: "GND"
- board text added: "H"
- board text added: "I"
- board text added: "ICSP"
- board text added: "ISO Enter"
- board text added: "ISO-#"
- board text added: "ISO-Shift"
- board text added: "ISO-\"
- board text added: "Insert"
- board text added: "J"
- board text added: "JTAG"
- board text added: "K"
- board text added: "L"
- board text added: "L Shift"
- board text added: "Left"
- board text added: "M"
- board text added: "MISO"
- board text added: "MOSI"
- board text added: "N"
- board text added: "O"
- board text added: "P"
- board text added: "PC6"
- board text added: "Page Down"
- board text added: "Page Up"
- board text added: "Period"
- board text added: "Q"
- board text added: "R"
- board text added: "R Shift"
- board text added: "RST"
- board text added: "Right"
- board text added: "S"
- board text added: "SCK"
- board text added: "T"
- board text added: "TCK"
- board text added: "TDI"
- board text added: "TDO"
- board text added: "TMS"
- board text added: "Tab"
- board text added: "U"
- board text added: "Up"
- board text added: "V"
- board text added: "VREF"
- board text added: "W"
- board text added: "X"
- board text added: "Y"
- board text added: "Z"
- board text added: "["
- board text added: "\"
- board text added: "]"
