File: a1800-compat/a1800-compat.kicad_pcb (KiCad board)
At the start: 2 copper layers, 371.5 x 137.8 mm, 255 parts, among them P1 USB_B, P2 CONN_02X03, SW1 SW_PUSH, U1 AT90USB1286, Y1 16Mhz

Commit message: Updating the 1800 board, adding a couple of related proects
Parts:
- added C10, C15: 1µF, Capacitors_SMD:C_0805_HandSoldering, F.Cu at (214.3, 166.9)
- added C11, C12, C13, C14: 0.1µF, Capacitors_SMD:C_0805_HandSoldering, F.Cu at (214.3, 166.9)
- added P3: CONN_02X05, Pin_Headers:Pin_Header_Straight_2x05, F.Cu at (266.7, 47.6)
- added R10, R12: 30kΩ, Resistors_SMD:R_0805_HandSoldering, F.Cu at (214.3, 166.9)
- added R11, R9: 10kΩ, Resistors_SMD:R_0805_HandSoldering, F.Cu at (214.3, 166.9)
- added REF**: GND Via, Keyboard:GNDVia-wRing, F.Cu at (286.0, 48.0)
- added REF**: GND Via, Keyboard:GNDVia-wRing, F.Cu at (281.1, 48.0)
- added U2: IS31FL3731, Housings_SSOP:SSOP-28_5.3x10.2mm_Pitch0.65mm, B.Cu at (317.1, 75.4)
- added U3: IS31FL3731, Housings_SSOP:SSOP-28_5.3x10.2mm_Pitch0.65mm, F.Cu at (168.8, 175.4)
- D1, D10, D101, D102, D104 (x2), D108, D109, D11, D111, D112, D113, D114, D115, D12, D13, D14, D15, D16, D17, D18, D19, D2, D20, D21, D22, D23, D24, D25, D26, D27, D28, D29, D3, D30, D31, D32, D33, D34, D35, D36, D37, D38, D39, D4, D40, D41, D42, D43, D44, D45, D46, D47, D48, D49, D5, D50, D51, D52, D53, D55, D56, D57, D58, D59, D6, D61, D62, D63, D64, D65, D66, D67, D68, D69, D7, D70, D71, D72, D74, D75, D76, D77, D78, D8, D80, D81, D82, D83, D84, D85, D86, D87, D88, D89, D9, D90, D91, D92, D93, D94, D95, D96, D97, D99: footprint Diodes_SMD:SOD-123 -> Keyboard:SOD-80
- moved P2 16.1 mm to (326.0, 15.5)
- moved C6 10.1 mm to (300.4, 33.0), turned to 90 degrees
- moved C7 4.32 mm to (298.3, 33.0), turned to 270 degrees
- moved C8 1.62 mm to (296.3, 33.0), turned to 90 degrees
- moved C9 0.90 mm to (284.6, 39.8), turned to 0 degrees
- moved C4 0.63 mm to (284.3, 48.0)
- moved C5 0.63 mm to (282.1, 48.0)
- moved R7 0.58 mm to (314.6, 33.0)
- moved R8 0.24 mm to (316.7, 33.0)
Connections:
- SW_100 pad SW1: Net-(D101-Pad2) -> Net-(D99-Pad2)
- SW_105 pad SW1: Net-(D104-Pad2) -> C11
- SW_105 pad SW2: C11 -> Net-(D104-Pad2)
- U1 pad 35: Net-(U1-Pad35) -> C14
- U1 pad 36: Net-(U1-Pad36) -> C15
- U1 pad 37: Net-(U1-Pad37) -> C16
- U1 pad 38: Net-(U1-Pad38) -> C17
- U1 pad 39: Net-(U1-Pad39) -> C18
- U1 pad 54: C18 -> TDI
- U1 pad 55: C17 -> TDO
- U1 pad 56: C16 -> TMS
- U1 pad 57: C15 -> TCK
- U1 pad 58: C14 -> Net-(U1-Pad58)
Routing:
- net SW_B2: track 254.5 -> 317.7 mm, vias 2 -> 3
- net SW_B8: track 307.7 -> 360.2 mm, vias 1 -> 2
- net SW_B7: track 332.3 -> 365.8 mm, vias 2 -> 3
- net MOSI: track 31.9 -> 0.00 mm
- net SW_B5: track 316.2 -> 347.5 mm, vias 1 -> 2
- net MISO: track 28.5 -> 0.00 mm, vias 1 -> 0
- net TCK: track 0.00 -> 28.1 mm
- net SW_B3: track 305.4 -> 332.9 mm, vias 1 -> 2
- net C18: track 253.3 -> 231.0 mm, vias 3 -> 1
- net C16: track 241.7 -> 219.3 mm, vias 3 -> 1
- net TDO: track 0.00 -> 22.3 mm
- net C15: track 200.7 -> 178.8 mm, vias 4 -> 2
- net TMS: track 0.00 -> 19.9 mm
- net +5V: track 115.6 -> 96.1 mm, vias 3 -> 2
- net C17: track 222.4 -> 203.2 mm, vias 3 -> 1
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Other:
- net class 10m: clearance 0.2032 -> 0.1905
- net class 8m added: clearance 0.1905, trace_width 0.2032, via_dia 0.6858, via_drill 0.3302
- net class Default: clearance 0.2032 -> 0.1905
- net class LED: clearance 0.2032 -> 0.1905
- net class Matrix: trace_width 0.254 -> 0.2032
- rule trace_clearance: 0.2032 -> 0.1905
