File: a1800-compat/a1800-compat.sch (KiCad schematic (older format))
At the start: 243 parts, among them P1 USB_B, P2 CONN_02X03, SW1 SW_PUSH, U1 AT90USB1286, Y1 16Mhz

Commit message: Updating the 1800 board, adding a couple of related proects
Parts:
- added P3: CONN_02X05, Pin_Headers:Pin_Header_Straight_2x05, symbol CONN_02X05
Connections:
- net +5V: now also P3.2 (P2)
- net C14: now also U1.35 ((A8)PC0); no longer U1.58 ((ADC3)PF3)
- net C15: now also U1.36 ((A9)PC1); no longer U1.57 ((ADC4/TCK)PF4)
- net C16: now also U1.37 ((A10)PC2); no longer U1.56 ((ADC5/TMS)PF5)
- net C17: now also U1.38 ((A11/T.3)PC3); no longer U1.55 ((ADC6/TDO)PF6)
- net C18: now also U1.39 ((A12/OC.3C)PC4); no longer U1.54 ((ADC7/TDI)PF7)
- net GND: now also P3.10 (P10), P3.4 (P4)
- net RESET: now also P3.6 (P6)
- new net TCK: P3.1 (P1), U1.57 ((ADC4/TCK)PF4)
- new net TDI: P3.9 (P9), U1.54 ((ADC7/TDI)PF7)
- new net TDO: P3.3 (P3), U1.55 ((ADC6/TDO)PF6)
- new net TMS: P3.5 (P5), U1.56 ((ADC5/TMS)PF5)
Changed lines of the file:
@@
 	6850 9100 6850 8900
 Wire Wire Line
-	7650 9250 7650 8900
+	7650 8900 7650 9250
 Wire Wire Line
 	7900 9250 7900 9100
@@
 Text GLabel 9200 13300 2    60   Input ~ 0
 C13
-Text GLabel 9200 13400 2    60   Input ~ 0
+Text GLabel 9200 10400 2    60   Input ~ 0
 C14
-Text GLabel 9200 13500 2    60   Input ~ 0
+Text GLabel 9200 10500 2    60   Input ~ 0
 C15
-Text GLabel 9200 13600 2    60   Input ~ 0
+Text GLabel 9200 10600 2    60   Input ~ 0
 C16
-Text GLabel 9200 13700 2    60   Input ~ 0
+Text GLabel 9200 10700 2    60   Input ~ 0
 C17
-Text GLabel 9200 13800 2    60   Input ~ 0
+Text GLabel 9200 10800 2    60   Input ~ 0
 C18
 Text GLabel 9200 11500 2    60   Input ~ 0
@@
 Wire Wire Line
 	12400 9200 12400 9000
+Text GLabel 9200 13500 2    60   Input ~ 0
+TCK
+Text GLabel 9200 13700 2    60   Input ~ 0
+TDO
+Text GLabel 9200 13600 2    60   Input ~ 0
+TMS
+Text GLabel 9200 13800 2    60   Input ~ 0
+TDI
+$Comp
+L CONN_02X05 P3
+U 1 1 5860B280
+P 1750 11600
+F 0 "P3" H 1750 11900 50  0000 C CNN
+F 1 "CONN_02X05" H 1750 11300 50  0000 C CNN
+F 2 "Pin_Headers:Pin_Header_Straight_2x05" H 1750 10400 50  0001 C CNN
+F 3 "" H 1750 10400 50  0000 C CNN
+	1    1750 11600
+	1    0    0    -1
+$EndComp
+Text GLabel 2400 11600 2    60   Input ~ 0
+RESET
+$Comp
+L +5V #PWR017
+U 1 1 58610ED6
+P 2200 11300
+F 0 "#PWR017" H 2200 11150 50  0001 C CNN
+F 1 "+5V" H 2200 11440 50  0000 C CNN
+F 2 "" H 2200 11300 50  0000 C CNN
+F 3 "" H 2200 11300 50  0000 C CNN
+	1    2200 11300
+	1    0    0    -1
+$EndComp
+Wire Wire Line
+	2000 11400 2200 11400
+Wire Wire Line
+	2200 11400 2200 11300
+Wire Wire Line
+	2000 11600 2400 11600
+Wire Wire Line
+	2000 11500 2100 11500
+Wire Wire Line
+	2100 11500 2100 12000
+Wire Wire Line
+	2100 11800 2000 11800
+$Comp
+L GND #PWR018
+U 1 1 58611DC2
+P 2100 12000
+F 0 "#PWR018" H 2100 11750 50  0001 C CNN
+F 1 "GND" H 2100 11850 50  0000 C CNN
+F 2 "" H 2100 12000 50  0000 C CNN
+F 3 "" H 2100 12000 50  0000 C CNN
+	1    2100 12000
+	1    0    0    -1
+$EndComp
+Connection ~ 2100 11800
+Text GLabel 1500 11400 0    60   Input ~ 0
+TCK
+Text GLabel 1500 11500 0    60   Input ~ 0
+TDO
+Text GLabel 1500 11600 0    60   Input ~ 0
+TMS
+Text GLabel 1500 11800 0    60   Input ~ 0
+TDI
 $EndSCHEMATC
