File: 1800-controller/1800-controller.kicad_pcb (KiCad board)
At the start: 2 copper layers, 100 x 45 mm, 63 parts, among them IC1 ATTINY45-S, P1 USB_OTG, P2 USB_A, P3 CONN_01X08, U1 TPS76333, U2 TUSB2036, U3 TPS2041B, Y1 Crystal_GND3

Commit message: Various updates I forgot to commit previously
Parts:
- added REF**: GND Via, Keyboard:GNDVia-wRing, F.Cu at (139.8, 46.2)
- added REF**: GND Via, Keyboard:GNDVia-wRing, F.Cu at (168.5, 57.0)
- added REF**: GND Via, Keyboard:GNDVia-wRing, F.Cu at (167.0, 64.5)
- added REF**: GND Via, Keyboard:GNDVia-wRing, F.Cu at (163.8, 46.2)
- added REF**: GND Via, Keyboard:GNDVia-wRing, F.Cu at (147.5, 46.2)
- added REF**: GND Via, Keyboard:GNDVia-wRing, F.Cu at (134.8, 61.5)
- added REF**: MountingHole_5mm, Mounting_Holes:MountingHole_5mm, F.Cu at (105.0, 58.0)
- added REF**: MountingHole_2.2mm_M2_ISO7380_Pad, Mounting_Holes:MountingHole_2.2mm_M2_ISO7380_Pad, F.Cu at (133.5, 50.0)
- added REF**: MountingHole_2.2mm_M2_ISO7380_Pad, Mounting_Holes:MountingHole_2.2mm_M2_ISO7380_Pad, F.Cu at (188.5, 50.0)
- added REF**: GND Via, Keyboard:GNDVia-wRing, F.Cu at (156.5, 67.2)
- added REF**: GND Via, Keyboard:GNDVia-wRing, F.Cu at (141.0, 67.5)
- added REF**: GND Via, Keyboard:GNDVia-wRing, F.Cu at (151.0, 61.0)
- added REF**: GND Via, Keyboard:GNDVia-wRing, F.Cu at (138.0, 53.5)
- added REF**: GND Via, Keyboard:GNDVia-wRing, F.Cu at (155.5, 54.5)
- added REF**: MountingHole_2.2mm_M2_ISO7380_Pad, Mounting_Holes:MountingHole_2.2mm_M2_ISO7380_Pad, F.Cu at (133.5, 75.0)
- added REF**: MountingHole_2.2mm_M2_ISO7380_Pad, Mounting_Holes:MountingHole_2.2mm_M2_ISO7380_Pad, F.Cu at (188.5, 75.0)
- added REF**: GND Via, Keyboard:GNDVia-wRing, F.Cu at (149.8, 56.0)
- IC1: footprint Housings_SOIC:SOIC-8_3.9x4.9mm_Pitch1.27mm -> Housings_SOIC:SOIJ-8_5.3x5.3mm_Pitch1.27mm
- P3: footprint Connectors_Molex:Molex_PicoBlade_53261-0871_08x1.25mm_Angled -> Connectors_Molex:Molex_PicoBlade_53048-0810_08x1.25mm_Angled
- moved P3 3.35 mm to (184.0, 69.0)
- moved C27 2.60 mm to (141.3, 76.2)
- moved IC1 2.60 mm to (143.1, 72.5)
Connections:
- P3 pad 1: +5V -> MOSI
- P3 pad 2: GND -> MISO
- P3 pad 3: MOSI -> SCK
- P3 pad 4: MISO -> RESET
- P3 pad 5: SCK -> GND
- P3 pad 6: RESET -> D2D-
- P3 pad 7: D2D- -> D2D+
- P3 pad 8: D2D+ -> +5V
Routing:
- net +5V: track 128.3 -> 142.5 mm
- net MOSI: track 45.0 -> 39.5 mm, vias 2 -> 0
- net MISO: track 45.4 -> 40.2 mm, vias 2 -> 0
- net SCK: track 45.9 -> 40.9 mm, vias 2 -> 0
- net D2D+: track 20.2 -> 22.9 mm
- net D2D-: track 21.0 -> 23.4 mm
- net Net-(IC1-Pad2): track 5.65 -> 7.51 mm
- net GND: track 11.5 -> 9.66 mm, vias 3 -> 2
- net RESET: track 51.1 -> 49.4 mm
- net Net-(IC1-Pad3): track 6.95 -> 8.21 mm
Other:
- outline, holes or cut-outs redrawn
- board text added: "USB Hub/ISP/Controller RevA"
- board text removed: "RevA"
- board text removed: "USB Hub/ISP/Controller"
