File: 1800-controller/1800-controller.sch (KiCad schematic (older format))
At the start: 63 parts, among them IC1 ATTINY45-S, P1 USB_OTG, P2 USB_A, P3 CONN_01X08, U1 TPS76333, U2 TUSB2036, U3 TPS2041B, Y1 Crystal_GND3

Commit message: Various updates I forgot to commit previously
Parts:
- IC1: footprint Housings_SOIC:SOIC-8_3.9x4.9mm_Pitch1.27mm -> Housings_SOIC:SOIJ-8_5.3x5.3mm_Pitch1.27mm
- R21, R3: footprint Resistors_SMD:R_0805_HandSoldering -> Resistors_SMD:R_0603_HandSoldering
- U3: symbol TPS2041B -> TPS2041B-RESCUE-1800-controller
Connections:
- net +5V: now also P3.8 (P8); no longer P3.1 (P1)
- net D2D+: now also P3.7 (P7); no longer P3.8 (P8)
- net D2D-: now also P3.6 (P6); no longer P3.7 (P7)
- net GND: now also P3.5 (P5); no longer P3.2 (P2)
- net MISO: now also P3.2 (P2); no longer P3.4 (P4)
- net MOSI: now also P3.1 (P1); no longer P3.3 (P3)
- net RESET: now also P3.4 (P4); no longer P3.6 (P6)
- net SCK: now also P3.3 (P3); no longer P3.5 (P5)
Other:
- moved on the sheet: P3
Changed lines of the file:
@@
 EESchema Schematic File Version 2
+LIBS:1800-controller-rescue
 LIBS:power
 LIBS:device
@@
 F 0 "R3" V 3880 1550 50  0000 C CNN
 F 1 "1.5k" V 3800 1550 50  0000 C CNN
-F 2 "Resistors_SMD:R_0805_HandSoldering" V 3730 1550 50  0001 C CNN
+F 2 "Resistors_SMD:R_0603_HandSoldering" V 3730 1550 50  0001 C CNN
 F 3 "" H 3800 1550 50  0000 C CNN
 	1    3800 1550
@@
 F 0 "IC1" H 8300 1750 50  0000 C CNN
 F 1 "ATTINY45-S" H 10450 950 50  0000 C CNN
-F 2 "Housings_SOIC:SOIC-8_3.9x4.9mm_Pitch1.27mm" H 10400 1350 50  0000 C CIN
+F 2 "Housings_SOIC:SOIJ-8_5.3x5.3mm_Pitch1.27mm" H 10400 1350 50  0000 C CIN
 F 3 "" H 9450 1350 50  0000 C CNN
 	1    9450 1350
@@
 F 0 "R21" V 7700 1000 50  0000 C CNN
 F 1 "1.7k" V 7600 1050 50  0000 C CNN
-F 2 "Resistors_SMD:R_0805_HandSoldering" V 7530 1050 50  0001 C CNN
+F 2 "Resistors_SMD:R_0603_HandSoldering" V 7530 1050 50  0001 C CNN
 F 3 "" H 7600 1050 50  0000 C CNN
 	1    7600 1050
@@
 L CONN_01X08 P3
 U 1 1 5867D3B0
-P 10400 3100
-F 0 "P3" H 10400 3550 50  0000 C CNN
-F 1 "CONN_01X08" V 10500 3100 50  0000 C CNN
-F 2 "Connectors_Molex:Molex_PicoBlade_53261-0871_08x1.25mm_Angled" H 10400 3100 50  0001 C CNN
-F 3 "" H 10400 3100 50  0000 C CNN
-	1    10400 3100
-	1    0    0    -1
+P 10600 3150
+F 0 "P3" H 10600 3600 50  0000 C CNN
+F 1 "CONN_01X08" V 10700 3150 50  0000 C CNN
+F 2 "Connectors_Molex:Molex_PicoBlade_53261-0871_08x1.25mm_Angled" H 10600 3150 50  0001 C CNN
+F 3 "" H 10600 3150 50  0000 C CNN
+	1    10600 3150
+	1    0    0    1
 $EndComp
 $Comp
 L +5V #PWR021
 U 1 1 5867E10B
-P 10100 2650
-F 0 "#PWR021" H 10100 2500 50  0001 C CNN
-F 1 "+5V" H 10100 2790 50  0000 C CNN
-F 2 "" H 10100 2650 50  0000 C CNN
-F 3 "" H 10100 2650 50  0000 C CNN
-	1    10100 2650
+P 10300 2700
+F 0 "#PWR021" H 10300 2550 50  0001 C CNN
+F 1 "+5V" H 10300 2840 50  0000 C CNN
+F 2 "" H 10300 2700 50  0000 C CNN
+F 3 "" H 10300 2700 50  0000 C CNN
+	1    10300 2700
 	1    0    0    -1
 $EndComp
@@
 L GND #PWR022
 U 1 1 5867E1D0
-P 9700 2950
-F 0 "#PWR022" H 9700 2700 50  0001 C CNN
-F 1 "GND" H 9700 2800 50  0000 C CNN
-F 2 "" H 9700 2950 50  0000 C CNN
-F 3 "" H 9700 2950 50  0000 C CNN
-	1    9700 2950
-	1    0    0    -1
-$EndComp
-Text GLabel 10200 3450 0    60   Input ~ 0
+P 9900 3700
+F 0 "#PWR022" H 9900 3450 50  0001 C CNN
+F 1 "GND" H 9900 3550 50  0000 C CNN
+F 2 "" H 9900 3700 50  0000 C CNN
+F 3 "" H 9900 3700 50  0000 C CNN
+	1    9900 3700
+	1    0    0    -1
+$EndComp
+Text GLabel 10400 2900 0    60   Input ~ 0
 D2D+
-Text GLabel 10200 3350 0    60   Input ~ 0
+Text GLabel 10400 3000 0    60   Input ~ 0
 D2D-
-Text GLabel 10200 3250 0    60   Input ~ 0
+Text GLabel 10400 3200 0    60   Input ~ 0
 RESET
-Text GLabel 10200 3150 0    60   Input ~ 0
+Text GLabel 10400 3300 0    60   Input ~ 0
 SCK
-Text GLabel 10200 3050 0    60   Input ~ 0
+Text GLabel 10400 3400 0    60   Input ~ 0
 MISO
-Text GLabel 10200 2950 0    60   Input ~ 0
+Text GLabel 10400 3500 0    60   Input ~ 0
 MOSI
-Wire Wire Line
-	10200 2850 9700 2850
-Wire Wire Line
-	9700 2850 9700 2950
-Wire Wire Line
-	10200 2750 10100 2750
-Wire Wire Line
-	10100 2750 10100 2650
 $Comp
 L Ferrite_Bead_Small L1
@@
 Connection ~ 7350 4800
 $Comp
-L TPS2041B U3
+L TPS2041B-RESCUE-1800-controller U3
 U 1 1 586703A8
 P 7950 5000
@@
 	0    1    1    0
 $EndComp
+Wire Wire Line
+	10400 2800 10300 2800
+Wire Wire Line
+	10300 2800 10300 2700
+Wire Wire Line
+	10400 3100 9900 3100
+Wire Wire Line
+	9900 3100 9900 3700
 $EndSCHEMATC
