File: isp/isp.kicad_pcb (KiCad board)
At the start: 2 copper layers, 38.1 x 20.3 mm, 17 parts, among them IC1 ATTINY45-S, P1 USB_OTG, P2 CONN_02X03

Commit message: Various updates I forgot to commit previously
Parts:
- removed the REF** at (93.3, 41.9)
- removed the REF** at (87.6, 45.7)
- removed the REF** at (107.3, 58.4)
- added REF**: GND Via, Keyboard:GNDVia-wRing, F.Cu at (96.5, 52.7)
- added REF**: GND Via, Keyboard:GNDVia-wRing, F.Cu at (85.7, 43.2)
- C1: footprint Capacitors_SMD:C_0805_HandSoldering -> Capacitors_SMD:C_0603_HandSoldering
- D1, D2: footprint Diodes_SMD:SOD-123 -> Diodes_SMD:SOD-323_HandSoldering
- IC1: footprint Housings_SOIC:SOIC-8_3.9x4.9mm_Pitch1.27mm -> Housings_SOIC:SOIJ-8_5.3x5.3mm_Pitch1.27mm
- R1, R2, R3: footprint Resistors_SMD:R_0805_HandSoldering -> Resistors_SMD:R_0603_HandSoldering
- moved R1 9.39 mm to (86.8, 47.0), turned to 180 degrees
- moved D2 8.37 mm to (83.8, 48.5)
- moved R3 7.75 mm to (86.8, 49.7), turned to 180 degrees
- moved REF** 7.62 mm to (85.7, 58.4)
- moved C1 3.74 mm to (88.8, 43.7), turned to 90 degrees
- moved IC1 3.44 mm to (93.0, 49.0), turned to 90 degrees
- moved D1 3.22 mm to (83.8, 52.5), turned to 270 degrees
- moved R2 2.72 mm to (86.8, 51.2), turned to 180 degrees
Routing:
- net D-: track 19.5 -> 9.65 mm, vias 2 -> 0
- net +5V: track 37.3 -> 29.8 mm, vias 2 -> 0
- net GND: track 2.89 -> 9.70 mm
- net MOSI: track 7.24 -> 12.6 mm
- net MISO: track 4.18 -> 9.49 mm
- net D+: track 9.52 -> 6.96 mm
- net SCK: track 9.41 -> 11.8 mm
- net RST: track 13.8 -> 11.7 mm
- net Net-(IC1-Pad3): track 8.28 -> 7.23 mm
- net Net-(IC1-Pad2): track 5.26 -> 6.25 mm
Other:
- net class Default: clearance 0.2 -> 0.1778; trace_width 0.25 -> 0.1778; via_dia 0.6 -> 0.6858; via_drill 0.4 -> 0.3302
- rule trace_clearance: 0.2 -> 0.1778
- rule trace_min: 0.2 -> 0.1778
- rule via_min_drill: 0.3 -> 0.3302
- rule via_min_size: 0.4 -> 0.6858
- board text added: "Tiny ISP RevB"
- board text removed: "Tiny ISP"
