File: isp/isp.sch (KiCad schematic (older format))
At the start: 10 parts, among them IC1 ATTINY85-S, P1 USB_OTG, P2 CONN_02X03

Commit message: Various updates I forgot to commit previously
Parts:
- D1, D2: footprint Diodes_SMD:SOD-123 -> Diodes_SMD:SOD-323_HandSoldering
- IC1: footprint Housings_SOIC:SOIC-8_3.9x4.9mm_Pitch1.27mm -> Housings_SOIC:SOIJ-8_5.3x5.3mm_Pitch1.27mm
Changed lines of the file:
@@
 LIBS:contrib
 LIBS:valves
+LIBS:Zilog
 LIBS:isp-cache
 EELAYER 25 0
@@
 F 0 "IC1" H 4100 2850 50  0000 C CNN
 F 1 "ATTINY85-S" H 6250 2050 50  0000 C CNN
-F 2 "Housings_SOIC:SOIC-8_3.9x4.9mm_Pitch1.27mm" H 6200 2450 50  0000 C CIN
+F 2 "Housings_SOIC:SOIJ-8_5.3x5.3mm_Pitch1.27mm" H 6200 2450 50  0001 C CIN
 F 3 "" H 5250 2450 50  0000 C CNN
 F 4 "556-ATTINY45-20SU" H 5250 2450 60  0001 C CNN "Mouser"
@@
 F 0 "D1" H 1900 3000 50  0000 C CNN
 F 1 "3.6v" H 1900 2800 50  0000 C CNN
-F 2 "Diodes_SMD:SOD-123" H 1900 2900 50  0001 C CNN
+F 2 "Diodes_SMD:SOD-323_HandSoldering" H 1900 2900 50  0001 C CNN
 F 3 "" H 1900 2900 50  0000 C CNN
 F 4 "621-BZT52C3V6-F" H 1900 2900 60  0001 C CNN "Mouser"
@@
 F 0 "D2" H 2200 3000 50  0000 C CNN
 F 1 "3.6v" H 2200 2800 50  0000 C CNN
-F 2 "Diodes_SMD:SOD-123" H 2200 2900 50  0001 C CNN
+F 2 "Diodes_SMD:SOD-323_HandSoldering" H 2200 2900 50  0001 C CNN
 F 3 "" H 2200 2900 50  0000 C CNN
 F 4 "621-BZT52C3V6-F" H 2200 2900 60  0001 C CNN "Mouser"
@@
 $EndComp
 $Comp
-L GND #PWR01
+L GND #PWR5
 U 1 1 5859EC1B
 P 1600 3300
-F 0 "#PWR01" H 1600 3050 50  0001 C CNN
+F 0 "#PWR5" H 1600 3050 50  0001 C CNN
 F 1 "GND" H 1600 3150 50  0000 C CNN
 F 2 "" H 1600 3300 50  0000 C CNN
@@
 $EndComp
 $Comp
-L GND #PWR02
+L GND #PWR4
 U 1 1 5859EC51
 P 1100 3000
-F 0 "#PWR02" H 1100 2750 50  0001 C CNN
+F 0 "#PWR4" H 1100 2750 50  0001 C CNN
 F 1 "GND" H 1100 2850 50  0000 C CNN
 F 2 "" H 1100 3000 50  0000 C CNN
@@
 	1600 2800 1600 3300
 $Comp
-L +5V #PWR03
+L +5V #PWR1
 U 1 1 5859EC8F
 P 1600 1900
-F 0 "#PWR03" H 1600 1750 50  0001 C CNN
+F 0 "#PWR1" H 1600 1750 50  0001 C CNN
 F 1 "+5V" H 1600 2040 50  0000 C CNN
 F 2 "" H 1600 1900 50  0000 C CNN
@@
 RST
 $Comp
-L +5V #PWR04
+L +5V #PWR2
 U 1 1 5859FDD9
 P 6700 2000
-F 0 "#PWR04" H 6700 1850 50  0001 C CNN
+F 0 "#PWR2" H 6700 1850 50  0001 C CNN
 F 1 "+5V" H 6700 2140 50  0000 C CNN
 F 2 "" H 6700 2000 50  0000 C CNN
@@
 $EndComp
 $Comp
-L GND #PWR05
+L GND #PWR3
 U 1 1 5859FE02
 P 6700 2900
-F 0 "#PWR05" H 6700 2650 50  0001 C CNN
+F 0 "#PWR3" H 6700 2650 50  0001 C CNN
 F 1 "GND" H 6700 2750 50  0000 C CNN
 F 2 "" H 6700 2900 50  0000 C CNN
@@
 MISO
 $Comp
-L GND #PWR06
+L GND #PWR7
 U 1 1 585A0230
 P 1900 4400
-F 0 "#PWR06" H 1900 4150 50  0001 C CNN
+F 0 "#PWR7" H 1900 4150 50  0001 C CNN
 F 1 "GND" H 1900 4250 50  0000 C CNN
 F 2 "" H 1900 4400 50  0000 C CNN
@@
 $EndComp
 $Comp
-L +5V #PWR07
+L +5V #PWR6
 U 1 1 585A0259
 P 1900 4000
-F 0 "#PWR07" H 1900 3850 50  0001 C CNN
+F 0 "#PWR6" H 1900 3850 50  0001 C CNN
 F 1 "+5V" H 1900 4140 50  0000 C CNN
 F 2 "" H 1900 4000 50  0000 C CNN
